File: hardware_design/pcb/dendrometer/sensor.brd (EAGLE design)
At the start: 35.6 x 61 mm, 23 parts, among them J1 AVR_SPI_PRG_6PTH, Q1 mosfet-N, U1 ATMEGA328P

Commit message: I've been way behind. Here is a shitload of stuff. Status is, everything is working pretty darn well right now
Parts:
- moved J1 51.4 mm to (6.99, 6.99)
- moved R5 39.8 mm to (6.99, 54.0), turned to 90 degrees
- moved PGRM 28.5 mm to (12.1, 33.0), turned to 90 degrees
- moved JP1 26.8 mm to (9.53, 26.7), turned to 90 degrees
- moved C4 26.8 mm to (29.5, 41.9), turned to 270 degrees
- moved C2 22.5 mm to (28.6, 55.2), turned to 180 degrees
- moved C5 21.6 mm to (6.99, 50.8), turned to 270 degrees
- moved R1 21.0 mm to (10.8, 19.1)
- moved R4 19.6 mm to (12.7, 29.8)
- moved C3 17.9 mm to (15.2, 34.9), turned to 90 degrees
- moved U$3 17.5 mm to (13.3, 24.1)
- moved R6 16.5 mm to (29.8, 51.4), turned to 270 degrees
- moved Q1 16.3 mm to (16.5, 31.1), turned to 90 degrees
- moved R3 15.3 mm to (17.1, 34.9), turned to 90 degrees
- moved R2 14.7 mm to (17.1, 21.6), turned to 270 degrees
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Connections:
- removed net N$8: LED1.C, U1.13
- new net N$5: LED1.C, U1.1
Routing:
- net V3.3: track 31.1 -> 106.9 mm
- net SDA: track 0.00 -> 49.4 mm, vias 0 -> 2
- net SCL: track 0.00 -> 46.5 mm, vias 0 -> 2
- net RST: track 29.0 -> 68.2 mm, vias 2 -> 0
- net N$5: track 0.00 -> 13.5 mm
- net TX: track 0.00 -> 13.5 mm
- net RX: track 0.00 -> 13.1 mm
- net SS: track 2.55 -> 13.5 mm
- net SENS_EN: track 0.00 -> 9.71 mm
- net N$8: track 9.62 -> 0.00 mm
- net N$3: track 0.00 -> 9.28 mm
- net N$10: track 0.00 -> 8.62 mm
- net VBAT: track 32.0 -> 39.0 mm
- net MOSI: track 19.9 -> 13.0 mm
- net N$2: track 0.00 -> 6.78 mm
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- added copper zone on layer 1, net GND
