File: hardware_design/pcb/dendrometer/sensor.sch (EAGLE design)
At the start: 23 parts, among them J1 AVR_SPI_PRG_6PTH, Q1 mosfet-N, U1 ATMEGA328P

Commit message: I've been way behind. Here is a shitload of stuff. Status is, everything is working pretty darn well right now
Connections:
- removed net N$8: LED1.C, U1.PB1(OC1A)
- new net N$5: LED1.C, U1.PD3(INT1)
Other:
- moved on the sheet: LED1, R6
Changed lines of the file:
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@@
 <instance part="R5" gate="G$1" x="45.72" y="175.26" rot="R90"/>
 <instance part="C4" gate="G$1" x="40.64" y="144.78" rot="R180"/>
-<instance part="LED1" gate="G$1" x="114.3" y="119.38" rot="R270"/>
-<instance part="R6" gate="G$1" x="119.38" y="127" rot="R270"/>
+<instance part="LED1" gate="G$1" x="121.92" y="137.16" rot="R270"/>
+<instance part="R6" gate="G$1" x="134.62" y="142.24" rot="R270"/>
 <instance part="PGRM" gate="G$1" x="27.94" y="83.82"/>
 <instance part="C5" gate="G$1" x="45.72" y="91.44" rot="R270"/>
@@
 <segment>
 <pinref part="R6" gate="G$1" pin="P$1"/>
-<wire x1="119.38" y1="132.08" x2="119.38" y2="134.62" width="0.1524" layer="91"/>
-<label x="119.38" y="134.62" size="1.778" layer="95"/>
+<wire x1="134.62" y1="147.32" x2="134.62" y2="149.86" width="0.1524" layer="91"/>
+<label x="139.7" y="149.86" size="1.778" layer="95"/>
 </segment>
 </net>
@@
 </segment>
 </net>
-<net name="N$8" class="0">
-<segment>
-<pinref part="U1" gate="G$1" pin="PB1(OC1A)"/>
-<wire x1="96.52" y1="119.38" x2="109.22" y2="119.38" width="0.1524" layer="91"/>
-<pinref part="LED1" gate="G$1" pin="C"/>
-</segment>
-</net>
 <net name="N$9" class="0">
 <segment>
 <pinref part="LED1" gate="G$1" pin="A"/>
-<wire x1="116.84" y1="119.38" x2="119.38" y2="119.38" width="0.1524" layer="91"/>
+<wire x1="124.46" y1="137.16" x2="134.62" y2="137.16" width="0.1524" layer="91"/>
 <pinref part="R6" gate="G$1" pin="P$2"/>
-<wire x1="119.38" y1="119.38" x2="119.38" y2="121.92" width="0.1524" layer="91"/>
 </segment>
 </net>
@@
 </segment>
 </net>
+<net name="N$5" class="0">
+<segment>
+<pinref part="U1" gate="G$1" pin="PD3(INT1)"/>
+<pinref part="LED1" gate="G$1" pin="C"/>
+<wire x1="96.52" y1="137.16" x2="116.84" y2="137.16" width="0.1524" layer="91"/>
+</segment>
+</net>
