File: hardware_design/pcb/dendrometer/sensor_sunstone.sch (EAGLE design)
At the start: 26 parts, among them Q2 PFET, U1 ATMEGA328P, U2 TPS61097-33, U3 MCP3425A0T-E/CH, U4 INDUCTORS_WURTH

Commit message: ....long time. bunch of stuff...oops
Parts:
- R3: value 1M -> 2M
- R4: value 6.8k -> DNP
- R7: value 43k -> 5.9k
Changed lines of the file:
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@@
 <setting verticaltext="up"/>
 </settings>
-<grid distance="0.1" unitdist="inch" unit="inch" style="lines" multiple="1" display="no" altdistance="0.01" altunitdist="inch" altunit="inch"/>
+<grid distance="0.1" unitdist="inch" unit="inch" style="lines" multiple="1" display="yes" altdistance="0.01" altunitdist="inch" altunit="inch"/>
 <layers>
 <layer number="1" name="Top" color="4" fill="1" visible="no" active="no"/>
@@
 <part name="C2" library="passives-7351" deviceset="CAPACITOR" device="0805-N" value="10uF"/>
 <part name="C3" library="passives-7351" deviceset="CAPACITOR" device="0603-N" value="0.1uF"/>
-<part name="R3" library="passives-7351" deviceset="RESISTOR" device="0603-N" value="1M"/>
+<part name="R3" library="passives-7351" deviceset="RESISTOR" device="0603-N" value="2M"/>
 <part name="ANT" library="SparkFun-Connectors" deviceset="M01" device="PTH"/>
 <part name="ICSP" library="SparkFun-Connectors" deviceset="AVR_SPI_PRG_6" device="PTH"/>
@@
 <part name="C6" library="passives-7351" deviceset="CAPACITOR" device="0603-N" value="0.1uF"/>
 <part name="C7" library="passives-7351" deviceset="CAPACITOR" device="0603-N" value="0.1uF"/>
-<part name="R4" library="passives-7351" deviceset="RESISTOR" device="0603-N" value="6.8k"/>
+<part name="R4" library="passives-7351" deviceset="RESISTOR" device="0603-N" value="DNP"/>
 <part name="SENS" library="SparkFun-Connectors" deviceset="M03" device="PTH"/>
-<part name="R7" library="passives-7351" deviceset="RESISTOR" device="0603-N" value="43k"/>
+<part name="R7" library="passives-7351" deviceset="RESISTOR" device="0603-N" value="5.9k"/>
 </parts>
 <sheets>
