File: hardware_design/pcb/dendrometer/sensor_v4.brd (EAGLE design)
At the start: 35.6 x 61 mm, 25 parts, among them J1 AVR_SPI_PRG_6PTH, Q2 MOSFET-PCHANNELIRLML2244, U1 ATMEGA328P

Commit message: bunch of shit. oops
Parts:
- R3: value 100k -> 1M
Changed lines of the file:
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@@
 <attribute name="NAME" x="19.52309375" y="42.555078125" size="1" layer="25" font="vector" ratio="11"/>
 </element>
-<element name="R3" library="passives-7351" package="R0603-N" value="100k" x="30.48" y="40.64" smashed="yes" rot="R90">
+<element name="R3" library="passives-7351" package="R0603-N" value="1M" x="30.48" y="40.64" smashed="yes" rot="R90">
 <attribute name="NAME" x="31.231921875" y="37.43009375" size="1" layer="25" font="vector" ratio="11" rot="R90"/>
 </element>
