File: hardware_design/pcb/dendrometer/sensor_v4.sch (EAGLE design)
At the start: 28 parts, among them J1 AVR_SPI_PRG_6PTH, Q2 MOSFET-PCHANNELIRLML2244, U1 ATMEGA328P

Commit message: made .brd for pcb fab house. and other minor code changes
Parts:
- removed J2: (no value), SparkFun-Connectors:M02PTH
- removed R10: 5.7-5.9k, passives-7351:RESISTOR0603-N
- removed SJ1: SOLDERJUMPERNC, SparkFun-Retired:SOLDERJUMPERNC
- R3: value 10k -> 100k
Connections:
- removed net +3V3/2: R4.P$1, SENS.3
- removed net N$3: C2.1, C7.1, J2.2, R10.P$1, SJ1.1, U$2.VOUT
- new net V-EXCITE: R4.P$1, SENS.3, U1.PC1(ADC1)
- net V3.3: now also C2.1, C7.1, U$2.VOUT; no longer J2.1, R10.P$2, SJ1.2
Changed lines of the file:
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@@
 <part name="C2" library="passives-7351" deviceset="CAPACITOR" device="0805-N" value="10uF"/>
 <part name="C3" library="passives-7351" deviceset="CAPACITOR" device="0603-N" value="0.1uF"/>
-<part name="R3" library="passives-7351" deviceset="RESISTOR" device="0603-N" value="10k"/>
+<part name="R3" library="passives-7351" deviceset="RESISTOR" device="0603-N" value="100k"/>
 <part name="JP2" library="SparkFun-Connectors" deviceset="M01" device="PTH"/>
 <part name="J1" library="SparkFun-Connectors" deviceset="AVR_SPI_PRG_6" device="PTH"/>
@@
 <part name="R4" library="passives-7351" deviceset="RESISTOR" device="0603-N" value="5.7-5.9k"/>
 <part name="SENS" library="SparkFun-Connectors" deviceset="M03" device="PTH"/>
-<part name="SJ1" library="SparkFun-Retired" deviceset="SOLDERJUMPER" device="NC"/>
-<part name="R10" library="passives-7351" deviceset="RESISTOR" device="0603-N" value="5.7-5.9k"/>
-<part name="J2" library="SparkFun-Connectors" deviceset="M02" device="PTH"/>
 </parts>
 <sheets>
@@
 <instance part="R4" gate="G$1" x="104.14" y="45.72" rot="R90"/>
 <instance part="SENS" gate="J$1" x="99.06" y="17.78"/>
-<instance part="SJ1" gate="1" x="73.66" y="30.48" rot="R180"/>
-<instance part="R10" gate="G$1" x="71.12" y="38.1" rot="R180"/>
-<instance part="J2" gate="G$1" x="71.12" y="48.26" rot="R270"/>
 </instances>
 <busses>
@@
 <pinref part="J1" gate="G$1" pin="6"/>
 <wire x1="38.1" y1="48.26" x2="55.88" y2="48.26" width="0.1524" layer="91"/>
-<label x="55.88" y="48.26" size="1.778" layer="95"/>
+<label x="50.8" y="48.26" size="1.778" layer="95"/>
 </segment>
 <segment>
@@
 <pinref part="J1" gate="G$1" pin="2"/>
 <wire x1="38.1" y1="53.34" x2="55.88" y2="53.34" width="0.1524" layer="91"/>
-<label x="55.88" y="53.34" size="1.778" layer="95"/>
+<label x="50.8" y="53.34" size="1.778" layer="95"/>
 </segment>
 <segment>
@@
 </segment>
 <segment>
-<pinref part="SJ1" gate="1" pin="2"/>
-<wire x1="68.58" y1="30.48" x2="63.5" y2="30.48" width="0.1524" layer="91"/>
-<wire x1="63.5" y1="30.48" x2="63.5" y2="38.1" width="0.1524" layer="91"/>
-<pinref part="R10" gate="G$1" pin="P$2"/>
-<wire x1="63.5" y1="38.1" x2="66.04" y2="38.1" width="0.1524" layer="91"/>
-<wire x1="63.5" y1="38.1" x2="63.5" y2="40.64" width="0.1524" layer="91"/>
-<junction x="63.5" y="38.1"/>
-<pinref part="J2" gate="G$1" pin="1"/>
-<wire x1="63.5" y1="40.64" x2="71.12" y2="40.64" width="0.1524" layer="91"/>
-<wire x1="63.5" y1="38.1" x2="55.88" y2="38.1" width="0.1524" layer="91"/>
-<label x="55.88" y="38.1" size="1.778" layer="95"/>
-<label x="55.88" y="38.1" size="1.778" layer="95"/>
+<pinref part="U$2" gate="TPS61097-33" pin="VOUT"/>
+<pinref part="C2" gate="G$1" pin="1"/>
+<wire x1="68.58" y1="20.32" x2="68.58" y2="10.16" width="0.1524" layer="91"/>
+<wire x1="68.58" y1="20.32" x2="78.74" y2="20.32" width="0.1524" layer="91"/>
+<junction x="68.58" y="20.32"/>
+<pinref part="C7" gate="G$1" pin="1"/>
+<wire x1="78.74" y1="20.32" x2="78.74" y2="10.16" width="0.1524" layer="91"/>
+<label x="76.2" y="20.32" size="1.778" layer="95"/>
 </segment>
 </net>
@@
 </segment>
 <segment>
-<label x="55.88" y="50.8" size="1.778" layer="95"/>
+<label x="50.8" y="50.8" size="1.778" layer="95"/>
 <wire x1="38.1" y1="50.8" x2="55.88" y2="50.8" width="0.1524" layer="91"/>
 <pinref part="J1" gate="G$1" pin="4"/>
@@
 </segment>
 </net>
-<net name="+3V3/2" class="0">
+<net name="V-EXCITE" class="0">
 <segment>
 <pinref part="R4" gate="G$1" pin="P$1"/>
@@
 <wire x1="111.76" y1="35.56" x2="104.14" y2="35.56" width="0.1524" layer="91"/>
 <wire x1="104.14" y1="35.56" x2="104.14" y2="40.64" width="0.1524" layer="91"/>
+<wire x1="111.76" y1="35.56" x2="116.84" y2="35.56" width="0.1524" layer="91"/>
+<junction x="111.76" y="35.56"/>
+<wire x1="116.84" y1="35.56" x2="116.84" y2="43.18" width="0.1524" layer="91"/>
+<label x="116.84" y="38.1" size="1.778" layer="95" rot="R90"/>
+</segment>
+<segment>
+<pinref part="U1" gate="G$1" pin="PC1(ADC1)"/>
+<wire x1="96.52" y1="165.1" x2="106.68" y2="165.1" width="0.1524" layer="91"/>
+<label x="99.06" y="165.1" size="1.778" layer="95"/>
 </segment>
 </net>
@@
 </segment>
 </net>
-<net name="N$3" class="0">
-<segment>
-<pinref part="U$2" gate="TPS61097-33" pin="VOUT"/>
-<pinref part="C2" gate="G$1" pin="1"/>
-<wire x1="68.58" y1="20.32" x2="68.58" y2="10.16" width="0.1524" layer="91"/>
-<wire x1="68.58" y1="20.32" x2="78.74" y2="20.32" width="0.1524" layer="91"/>
-<junction x="68.58" y="20.32"/>
-<pinref part="C7" gate="G$1" pin="1"/>
-<wire x1="78.74" y1="20.32" x2="78.74" y2="10.16" width="0.1524" layer="91"/>
-<wire x1="78.74" y1="20.32" x2="78.74" y2="30.48" width="0.1524" layer="91"/>
-<junction x="78.74" y="20.32"/>
-<pinref part="SJ1" gate="1" pin="1"/>
-<wire x1="78.74" y1="30.48" x2="78.74" y2="38.1" width="0.1524" layer="91"/>
-<junction x="78.74" y="30.48"/>
-<pinref part="R10" gate="G$1" pin="P$1"/>
-<wire x1="78.74" y1="38.1" x2="76.2" y2="38.1" width="0.1524" layer="91"/>
-<wire x1="78.74" y1="38.1" x2="78.74" y2="40.64" width="0.1524" layer="91"/>
-<junction x="78.74" y="38.1"/>
-<pinref part="J2" gate="G$1" pin="2"/>
-<wire x1="78.74" y1="40.64" x2="73.66" y2="40.64" width="0.1524" layer="91"/>
-</segment>
-</net>

Commit message: bunch of shit. oops
Parts:
- R3: value 100k -> 1M
Changed lines of the file:
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@@
 <part name="C2" library="passives-7351" deviceset="CAPACITOR" device="0805-N" value="10uF"/>
 <part name="C3" library="passives-7351" deviceset="CAPACITOR" device="0603-N" value="0.1uF"/>
-<part name="R3" library="passives-7351" deviceset="RESISTOR" device="0603-N" value="100k"/>
+<part name="R3" library="passives-7351" deviceset="RESISTOR" device="0603-N" value="1M"/>
 <part name="JP2" library="SparkFun-Connectors" deviceset="M01" device="PTH"/>
 <part name="J1" library="SparkFun-Connectors" deviceset="AVR_SPI_PRG_6" device="PTH"/>
