File: hardware_design/pcb/dendrometer/receiver_shield.brd (EAGLE design)
At the start: 70.2 x 57.5 mm, 24 parts, among them Q1 MFET-N, Q2 MFET-N, Q3 MFET-N, Q4 MFET-N, Q5 MFET-N

Commit message: bunch of shit. oops
Parts:
- added D1: (no value), SparkFun-LED:LED-0603
- added R11: 10k, passives-7351:R0603-N
- added R12: 440, passives-7351:R0603-N
Connections:
- new net N$1: D1.A, R12.2
- new net PIN_3: PCB1.3, R12.1
- new net PIN_5: JP1.8, PCB1.5, R11.1
- net 5V: now also R11.2
- net GND: now also D1.C
Routing:
- net PIN_5: track 0.00 -> 38.8 mm, vias 0 -> 2
- net 5V: track 119.6 -> 134.1 mm, vias 2 -> 4
- net PIN_3: track 0.00 -> 7.47 mm
- net N$1: track 0.00 -> 4.63 mm
- net PIN_4: track 41.6 -> 41.1 mm
Other:
- outline, holes or cut-outs redrawn

Commit message: ....long time. bunch of stuff...oops
Parts:
- removed U$3: LINX_2032BAT_HLDER, _my-parts:LINX_2032BAT_HLDER
- added U$2: 2032_BAT_HLDR, _my-parts:2032_BAT_HLDR_MPD
Connections:
- net GND: now also U$2.P$1; no longer U$3.P$1
- net N$2: now also U$2.P$2; no longer U$3.BAT_POS$1, U$3.BAT_POS$2, U$3.BAT_POS$3, U$3.BAT_POS$4
Routing:
- net N$2: track 46.1 -> 85.7 mm, vias 0 -> 1
- net PIN_4: track 41.1 -> 45.4 mm
- net PIN_5: track 38.8 -> 35.2 mm
- net GND: track 22.1 -> 24.7 mm
Other:
- outline, holes or cut-outs redrawn
