File: hardware_design/pcb/dendrometer/receiver_shield.sch (EAGLE design)
At the start: 24 parts, among them Q1 MFET-N, Q2 MFET-N, Q3 MFET-N, Q4 MFET-N, Q5 MFET-N

Commit message: bunch of shit. oops
Parts:
- added D1: (no value), SparkFun-LED:LED0603
- added R11: 10k, passives-7351:RESISTOR0603-N
- added R12: 440, passives-7351:RESISTOR0603-N
Connections:
- new net N$1: D1.A, R12.P$2
- new net PIN_3: PCB1.~3, R12.P$1
- new net PIN_5: JP1.CD, PCB1.~5, R11.P$1
- net 5V: now also R11.P$2
- net GND: now also D1.C
Changed lines of the file:
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@@
 <setting verticaltext="up"/>
 </settings>
-<grid distance="0.1" unitdist="inch" unit="inch" style="lines" multiple="1" display="no" altdistance="0.01" altunitdist="inch" altunit="inch"/>
+<grid distance="0.1" unitdist="inch" unit="inch" style="lines" multiple="1" display="yes" altdistance="0.01" altunitdist="inch" altunit="inch"/>
 <layers>
 <layer number="1" name="Top" color="4" fill="1" visible="no" active="no"/>
@@
 <part name="R9" library="passives-7351" deviceset="RESISTOR" device="0603-N" value="10k"/>
 <part name="R10" library="passives-7351" deviceset="RESISTOR" device="0603-N" value="10k"/>
+<part name="R11" library="passives-7351" deviceset="RESISTOR" device="0603-N" value="10k"/>
+<part name="D1" library="SparkFun-LED" deviceset="LED" device="0603"/>
+<part name="R12" library="passives-7351" deviceset="RESISTOR" device="0603-N" value="440"/>
 </parts>
 <sheets>
@@
 <instance part="R9" gate="G$1" x="312.42" y="83.82" rot="R90"/>
 <instance part="R10" gate="G$1" x="327.66" y="83.82" rot="R90"/>
+<instance part="R11" gate="G$1" x="81.28" y="96.52" rot="R90"/>
+<instance part="D1" gate="G$1" x="55.88" y="114.3" rot="R90"/>
+<instance part="R12" gate="G$1" x="45.72" y="114.3"/>
 </instances>
 <busses>
@@
 <wire x1="327.66" y1="88.9" x2="327.66" y2="93.98" width="0.1524" layer="91"/>
 <label x="327.66" y="93.98" size="1.778" layer="95" rot="R90" xref="yes"/>
+</segment>
+<segment>
+<pinref part="R11" gate="G$1" pin="P$2"/>
+<wire x1="81.28" y1="101.6" x2="81.28" y2="106.68" width="0.1524" layer="91"/>
+<label x="81.28" y="104.14" size="1.778" layer="95" rot="R90"/>
 </segment>
 </net>
@@
 <wire x1="53.34" y1="78.74" x2="53.34" y2="86.36" width="0.1524" layer="91"/>
 <label x="53.34" y="83.82" size="1.778" layer="95" rot="R90"/>
+</segment>
+<segment>
+<pinref part="D1" gate="G$1" pin="C"/>
+<wire x1="60.96" y1="114.3" x2="63.5" y2="114.3" width="0.1524" layer="91"/>
+<wire x1="63.5" y1="114.3" x2="63.5" y2="106.68" width="0.1524" layer="91"/>
+<label x="63.5" y="106.68" size="1.778" layer="95" rot="R180"/>
 </segment>
 </net>
@@
 </segment>
 </net>
+<net name="PIN_3" class="0">
+<segment>
+<pinref part="PCB1" gate="G$1" pin="~3"/>
+<wire x1="86.36" y1="78.74" x2="86.36" y2="86.36" width="0.1524" layer="91"/>
+<label x="86.36" y="81.28" size="1.778" layer="95" rot="R90"/>
+</segment>
+<segment>
+<pinref part="R12" gate="G$1" pin="P$1"/>
+<wire x1="40.64" y1="114.3" x2="35.56" y2="114.3" width="0.1524" layer="91"/>
+<label x="35.56" y="114.3" size="1.778" layer="95" rot="R180" xref="yes"/>
+</segment>
+</net>
+<net name="PIN_5" class="0">
+<segment>
+<wire x1="165.1" y1="127" x2="149.86" y2="127" width="0.1524" layer="91"/>
+<label x="149.86" y="127" size="1.778" layer="95"/>
+<pinref part="JP1" gate="G$1" pin="CD"/>
+</segment>
+<segment>
+<pinref part="PCB1" gate="G$1" pin="~5"/>
+<wire x1="81.28" y1="78.74" x2="81.28" y2="91.44" width="0.1524" layer="91"/>
+<label x="81.28" y="81.28" size="1.778" layer="95" rot="R90"/>
+<wire x1="81.28" y1="91.44" x2="78.74" y2="91.44" width="0.1524" layer="91"/>
+<pinref part="R11" gate="G$1" pin="P$1"/>
+<junction x="81.28" y="91.44"/>
+</segment>
+</net>
+<net name="N$1" class="0">
+<segment>
+<pinref part="D1" gate="G$1" pin="A"/>
+<pinref part="R12" gate="G$1" pin="P$2"/>
+<wire x1="50.8" y1="114.3" x2="53.34" y2="114.3" width="0.1524" layer="91"/>
+</segment>
+</net>

Commit message: ....long time. bunch of stuff...oops
Parts:
- removed U$3: LINX_2032BAT_HLDER, _my-parts:LINX_2032BAT_HLDER
- added U$2: 2032_BAT_HLDR, _my-parts:2032_BAT_HLDR
Connections:
- net GND: now also U$2.GND; no longer U$3.BAT_NEG
- net N$2: now also U$2.VBAT; no longer U$3.BAT_POS
Changed lines of the file:
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@@
 <setting verticaltext="up"/>
 </settings>
-<grid distance="0.1" unitdist="inch" unit="inch" style="lines" multiple="1" display="yes" altdistance="0.01" altunitdist="inch" altunit="inch"/>
+<grid distance="0.1" unitdist="inch" unit="inch" style="lines" multiple="1" display="no" altdistance="0.01" altunitdist="inch" altunit="inch"/>
 <layers>
 <layer number="1" name="Top" color="4" fill="1" visible="no" active="no"/>
@@
 <part name="PCB1" library="Arduino_revB" deviceset="ARDUINO_UNO" device=""/>
 <part name="U$1" library="_my-parts" deviceset="DS3231M" device=""/>
-<part name="U$3" library="_my-parts" deviceset="LINX_2032BAT_HLDER" device=""/>
 <part name="U$4" library="LowPowerLab" deviceset="RFM69" device=""/>
 <part name="Q1" library="SparkFun-DiscreteSemi" deviceset="MOSFET-NCHANNEL" device="AO3404A" value="MFET-N"/>
@@
 <part name="D1" library="SparkFun-LED" deviceset="LED" device="0603"/>
 <part name="R12" library="passives-7351" deviceset="RESISTOR" device="0603-N" value="440"/>
+<part name="U$2" library="_my-parts" deviceset="2032_BAT_HLDR" device=""/>
 </parts>
 <sheets>
@@
 <instance part="PCB1" gate="G$1" x="68.58" y="58.42"/>
 <instance part="U$1" gate="G$1" x="139.7" y="96.52"/>
-<instance part="U$3" gate="G$1" x="162.56" y="88.9"/>
 <instance part="U$4" gate="G$1" x="101.6" y="132.08"/>
 <instance part="Q1" gate="G$1" x="198.12" y="35.56" rot="R270"/>
@@
 <instance part="D1" gate="G$1" x="55.88" y="114.3" rot="R90"/>
 <instance part="R12" gate="G$1" x="45.72" y="114.3"/>
+<instance part="U$2" gate="G$1" x="162.56" y="88.9"/>
 </instances>
 <busses>
@@
 </segment>
 <segment>
-<pinref part="U$3" gate="G$1" pin="BAT_NEG"/>
-<wire x1="162.56" y1="83.82" x2="162.56" y2="78.74" width="0.1524" layer="91"/>
 <label x="162.56" y="78.74" size="1.778" layer="95"/>
+<pinref part="U$2" gate="G$1" pin="GND"/>
+<wire x1="162.56" y1="81.28" x2="162.56" y2="78.74" width="0.1524" layer="91"/>
 </segment>
 <segment>
@@
 <pinref part="U$1" gate="G$1" pin="VBAT"/>
 <wire x1="152.4" y1="96.52" x2="162.56" y2="96.52" width="0.1524" layer="91"/>
-<pinref part="U$3" gate="G$1" pin="BAT_POS"/>
 <wire x1="162.56" y1="96.52" x2="162.56" y2="93.98" width="0.1524" layer="91"/>
-</segment>
-</net>
+<pinref part="U$2" gate="G$1" pin="VBAT"/>
+</segment>
+</net>
