File: hardware_design/pcb/dendrometer/sensor_sunstone.brd (EAGLE design)
At the start: 35.6 x 39.4 mm, 26 parts, among them J1 AVR_SPI_PRG_6PTH, Q2 PFET, U1 ATMEGA328P, U2 TPS61097-33, U3 MCP3425A0T-E/CH

Commit message: generated gerber files and did some minor mech. work
Parts:
- removed J1: AVR_SPI_PRG_6PTH, SparkFun-Connectors:2X3
- removed JP2: M01PTH, SparkFun-Connectors:1X01
- removed U$4: INDUCTORS_WURTH, _my-parts:WURTH_10UH_650MA
- added ANT: M01PTH, SparkFun-Connectors:1X01
- added ICSP: AVR_SPI_PRG_6PTH, SparkFun-Connectors:2X3
- added U4: INDUCTORS_WURTH, _my-parts:WURTH_10UH_650MA
- moved C5 21.7 mm to (6.35, 26.7)
- moved R5 21.7 mm to (8.89, 26.7)
- moved U$5 21.7 mm to (20.8, 14.0)
- moved R4 21.6 mm to (30.0, 25.4)
- moved R7 21.6 mm to (33.0, 25.4)
- moved U3 21.6 mm to (30.5, 34.3)
- moved C4 21.6 mm to (25.4, 19.1)
- moved PGRM 21.6 mm to (10.2, 8.89)
- moved Q2 21.6 mm to (30.5, 21.6)
- moved R1 21.6 mm to (21.6, 30.5)
- moved R2 21.6 mm to (24.1, 30.5)
- moved U$1 21.6 mm to (17.8, 8.89)
- moved U1 21.6 mm to (19.1, 19.1)
- moved U2 21.6 mm to (16.5, 30.5)
- moved C1 21.6 mm to (16.5, 35.6)
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Connections:
- net GND: now also ICSP.6; no longer J1.6
- net MISO: now also ICSP.1; no longer J1.1
- net MOSI: now also ICSP.4; no longer J1.4
- net N$1: now also U4.P$1; no longer U$4.P$1
- net N$7: now also ANT.1; no longer JP2.1
- net RST: now also ICSP.5; no longer J1.5
- net SCK: now also ICSP.3; no longer J1.3
- net V3.3: now also ICSP.2; no longer J1.2
- net VBAT: now also U4.P$2; no longer U$4.P$2
Routing:
- net IRQ: track 8.84 -> 17.5 mm
- net V3.3: track 49.5 -> 54.8 mm
- net TX: track 12.5 -> 17.2 mm
- net VBAT: track 36.8 -> 39.4 mm
- net RX: track 23.6 -> 26.1 mm
- net SS: track 9.84 -> 12.2 mm
- net GND: track 4.59 -> 6.62 mm
- net SCK: track 28.5 -> 30.3 mm
- net RST: track 47.1 -> 48.7 mm
- net N$10: track 4.81 -> 6.30 mm
- net N$5: track 3.39 -> 1.90 mm
- net MOSI: track 20.7 -> 21.9 mm
- net N$9: track 2.05 -> 3.19 mm
- net MISO: track 23.2 -> 24.0 mm
- net N$2: track 4.45 -> 5.17 mm
Other:
- board text added: "U4"
- board text added: "dendro_v4 2016.04.11"

Commit message: bunch of shit. oops
Parts:
- R3: value 100k -> 1M
Changed lines of the file:
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@@
 <attribute name="NAME" x="23.33309375" y="27.823078125" size="1.016" layer="25" font="vector" ratio="16"/>
 </element>
-<element name="R3" library="passives-7351" package="R0603-N" value="100k" x="33.02" y="20.32" smashed="yes" rot="R90">
+<element name="R3" library="passives-7351" package="R0603-N" value="1M" x="33.02" y="20.32" smashed="yes" rot="R90">
 <attribute name="NAME" x="31.993921875" y="18.12609375" size="1.016" layer="25" font="vector" ratio="16" rot="R90"/>
 </element>

Commit message: ....long time. bunch of stuff...oops
Parts:
- R3: value 1M -> 2M
- R4: value 6.8k -> DNP
- R7: value 43k -> 5.9k
Changed lines of the file:
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@@
 <attribute name="NAME" x="23.33309375" y="27.823078125" size="1.016" layer="25" font="vector" ratio="16"/>
 </element>
-<element name="R3" library="passives-7351" package="R0603-N" value="1M" x="33.02" y="20.32" smashed="yes" rot="R90">
+<element name="R3" library="passives-7351" package="R0603-N" value="2M" x="33.02" y="20.32" smashed="yes" rot="R90">
 <attribute name="NAME" x="31.993921875" y="18.12609375" size="1.016" layer="25" font="vector" ratio="16" rot="R90"/>
 </element>
@@
 <attribute name="NAME" x="20.828" y="32.512" size="1.016" layer="25" font="vector" ratio="16"/>
 </element>
-<element name="R4" library="passives-7351" package="R0603-N" value="6.8k" x="29.972" y="25.4" smashed="yes" rot="R270">
+<element name="R4" library="passives-7351" package="R0603-N" value="DNP" x="29.972" y="25.4" smashed="yes" rot="R270">
 <attribute name="NAME" x="27.950078125" y="26.32390625" size="1.016" layer="25" font="vector" ratio="16" rot="R270"/>
 </element>
@@
 <attribute name="VALUE" x="34.29" y="32.385" size="1.27" layer="27" rot="R180"/>
 </element>
-<element name="R7" library="passives-7351" package="R0603-N" value="43k" x="33.02" y="25.4" smashed="yes" rot="R270">
+<element name="R7" library="passives-7351" package="R0603-N" value="5.9k" x="33.02" y="25.4" smashed="yes" rot="R270">
 <attribute name="NAME" x="32.374921875" y="24.60309375" size="1.016" layer="25" font="vector" ratio="16" rot="R90"/>
 </element>
