File: hardware_design/pcb/dendrometer/sensor_v5.brd (EAGLE design)
At the start: 35.6 x 61 mm, 27 parts, among them J1 AVR_SPI_PRG_6PTH, Q2 MOSFET-P, U1 ATMEGA328P, U2 LM4040A20IDBZT

Commit message: cleanup..
Parts:
- added R8: 330, passives-7351:R0603-N
- U$4: value INDUCTORS_WURTH -> 4.7uH
- moved U$5 30.8 mm to (18.8, 43.7), flipped to the bottom, turned to 0 degrees
- moved J1 27.7 mm to (5.84, 36.8)
- moved C5 19.1 mm to (32.5, 33.5), turned to 90 degrees
- moved JP2 19.0 mm to (14.2, 33.4)
- moved U1 15.9 mm to (11.4, 44.5), turned to 270 degrees
- moved C4 15.1 mm to (11.9, 37.8), turned to 180 degrees
- moved U$4 9.45 mm to (21.3, 53.5), turned to 270 degrees
- moved PGRM 7.40 mm to (17.5, 33.0), turned to 0 degrees
- moved C7 7.15 mm to (15.0, 56.1)
- moved LED1 7.11 mm to (14.2, 51.3)
- moved C6 6.90 mm to (20.3, 57.7)
- moved C2 6.43 mm to (13.0, 55.9)
- moved C1 6.12 mm to (22.4, 57.4)
- moved R6 5.14 mm to (11.3, 51.7), turned to 0 degrees
- moved SENS 4.60 mm to (27.4, 55.1)
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Connections:
- new net S_EN: Q2.3, R8.1
- net V_REF: now also R8.2; no longer Q2.3
Routing:
- net V3.3: track 174.2 -> 4.72 mm, vias 0 -> 1
- net GND: track 112.3 -> 19.4 mm, vias 0 -> 1
- net RST: track 68.8 -> 1.66 mm, vias 2 -> 0
- net SCK: track 51.8 -> 2.43 mm, vias 2 -> 0
- net MISO: track 37.6 -> 6.12 mm, vias 2 -> 0
- net IRQ: track 40.7 -> 15.9 mm, vias 2 -> 1
- net MOSI: track 35.4 -> 14.5 mm, vias 2 -> 0
- net RX: track 13.0 -> 23.3 mm
- net SENS_EN: track 15.9 -> 24.3 mm, vias 0 -> 2
- net N$10: track 10.2 -> 3.16 mm
- net VBAT: track 53.1 -> 59.5 mm
- net N$7: track 2.83 -> 8.34 mm
- net S_EN: track 0.00 -> 5.25 mm
- net SDA: track 12.9 -> 8.54 mm, vias 2 -> 0
- net V_REF: track 16.4 -> 13.8 mm
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- added copper zone on layer 16, net GND
- added copper zone on layer 1, net V3.3
- removed copper zone on layer 1, net GND
