File: sap-flux/hardware/pcb/MAX31855T_BREAKOUT.brd (EAGLE design)
At the start: 16.8 x 23.8 mm, 6 parts, among them U1 MAX31855K

Commit message: crazy long time since I did this. hah
Parts:
- C1: value (none) -> 0.1µF
- R1: value (none) -> 10k
Changed lines of the file:
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@@
 </autorouter>
 <elements>
-<element name="C1" library="passives-7351" package="C0805-L" value="" x="13.97" y="9.36625" rot="R270"/>
+<element name="C1" library="passives-7351" package="C0805-L" value="0.1µF" x="13.97" y="9.36625" rot="R270"/>
 <element name="GND" library="SparkFun-Connectors" package="1X05" value="" x="12.7" y="2.54" rot="R180"/>
-<element name="R1" library="passives-7351" package="R0603-N" value="" x="4.60375" y="13.335" rot="R90"/>
+<element name="R1" library="passives-7351" package="R0603-N" value="10k" x="4.60375" y="13.335" rot="R90"/>
 <element name="U1" library="SparkFun-AnalogIC" package="SOIC8" value="MAX31855K" x="8.89" y="11.43" rot="R180"/>
 <element name="T-" library="SparkFun-Connectors" package="LUXEON-PAD" value="" x="10.95375" y="19.84375" rot="R90"/>
