File: sap-flux/hardware/pcb/MAX31855T_BREAKOUT.sch (EAGLE design)
At the start: 6 parts, among them U1 MAX31855K

Commit message: crazy long time since I did this. hah
Parts:
- C1: value (none) -> 0.1µF
- R1: value (none) -> 10k
Changed lines of the file:
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@@
 <parts>
 <part name="U1" library="SparkFun-AnalogIC" deviceset="MAX31855K" device=""/>
-<part name="C1" library="passives-7351" deviceset="CAPACITOR" device="0805-L"/>
-<part name="R1" library="passives-7351" deviceset="RESISTOR" device="0603-N"/>
+<part name="C1" library="passives-7351" deviceset="CAPACITOR" device="0805-L" value="0.1µF"/>
+<part name="R1" library="passives-7351" deviceset="RESISTOR" device="0603-N" value="10k"/>
 <part name="GND" library="SparkFun-Connectors" deviceset="M05" device="PTH"/>
 <part name="T-" library="SparkFun-Connectors" deviceset="M01" device="SMD"/>
