File: sap-flux/hardware/pcb/sap_flux-v10.brd (EAGLE design)
At the start: 100 x 80 mm, 68 parts, among them J1 MF-CON-2.54mm-01x02, J2 MF-CON-2.54mm-01x02, J3 MF-CON-2.54mm-01x02, J4 KLDX-0202-B, Q1 MOSFET-PCHANNELSOT23-3, U1 MAX31856MUD+, U2 MAX31856MUD+, U3 MAX31856MUD+, U4 MCP73871, U5 ADP2503, U6 ADP1614

Commit message: sap flux BOM, Gerbers, Radiation Shield Files
Parts:
- added ANT1: ANTENNA-433_CHIP, My_RF:ANT_433_CHIP
- added C30, C31: 0.1uF, My_Passives:C0603-N
- added D6: green, My_LEDs:LED0603
- added D7: red, My_LEDs:LED0603
- added FRAME3: FRAME-LETTERNO_PACKAGE, My_Aesthetics:DUMMY
- added J5: CON_01X02TINY, My_Connectors:1X02_TINY
- added J6: (no value), My_Connectors:1X06
- added JP1: 1, My_Passives:PAD-JUMPER-2-NO_YES_SILK
- added JP2: 2, My_Passives:PAD-JUMPER-2-NO_YES_SILK
- added JP3: 4, My_Passives:PAD-JUMPER-2-NO_YES_SILK
- added LOGO1: OSHW-LOGOS-COPPER, My_Aesthetics:OSHW-LOGO-S_COPPER
- added Q2: battery reading nfet, My_Descrete_Semiconductors:SOT23-3
- added R19, R24: 10k, My_Passives:R0603-N
- added R20, R21: 1k, My_Passives:R0603-N
- added R22: 33k, My_Passives:R0603-N
- added R23: 68k, My_Passives:R0603-N
- added TC1: TC2030-IDC-NL, My_Connectors:TC2030-IDC-NL
- added U7: ATMEGA328P_32PIN-MU, My_IC_Digital:MLF32_RECTPADS
- added U8: RFM69HCW-433MHZ, My_RF:RFM69HCW-XXXS2
- added U9: WINBOND_FLASH_4MBIT-SOIC, My_IC_Digital:SOIC8
- added Y1: 8MHZ, My_xTal:RESONATOR-SMD
- BATT1: value BATTERY_HOLDER18650 -> BATTERY_HOLDER-18650_CLIP; device My_Connectors:BAT_18650-KEYSTONE-1043 -> My_Connectors:BAT_18650_CLIP
- C1, C14, C4, C5, C6: value 0.1uF -> 10uF; device My_Passives:C0603-N -> My_Passives:C0805-N
- C10: value 0.1uF -> 3300pF
- C11: value 0.1uF -> 4700uF; device My_Passives:C0603-N -> My_Passives:CP_TH_5MM
- C12, C13, C2, C3, C7: value 0.01uF -> 10uF; device My_Passives:C0603-N -> My_Passives:C0805-N
- C15: value 0.1uF -> 0.01uF
- C16: value 4700uF -> 0.1uF; device My_Passives:CP10MM -> My_Passives:C0603-N
- C17, C18, C20, C27: value 10uF -> 0.01uF; device My_Passives:C0805-N -> My_Passives:C0603-N
- C19, C21, C22, C26, C28, C29: value 10uF -> 0.1uF; device My_Passives:C0805-N -> My_Passives:C0603-N
- C23: value 22nF -> 0.1uF
- C24: value 33pF -> 0.1uF
- C25: value 47nF -> 0.01uF
- C8: value 0.01uF -> 4700pF
- C9: value 0.1uF -> 2200pF
- D1: value PMEG4005EJ -> (none); device My_Descrete_Semiconductors:SOD-323 -> My_LEDs:LED0603
- D4: value (none) -> DIODE-SCHOTTKY-SOD123FL; device My_LEDs:LED0603 -> My_Descrete_Semiconductors:SOD-123FL
- D5: value DIODE-SCHOTTKYSOD128 -> DIODE-SCHOTTKY-SOD128
- J1: value MF-CON-2.54mm-01x02 -> CON_01X02-0.2"_POL; device My_Connectors:PTH_2.54MM_01X02 -> My_Connectors:1X02_SCREWTERM_0.2IN
- J2, J3: value MF-CON-2.54mm-01x02 -> CON_01X02TINY; device My_Connectors:PTH_2.54MM_01X02 -> My_Connectors:1X02_TINY
- J4: value KLDX-0202-B -> CON_01X02TINY; device My_Connectors:DC_PWR_JACK -> My_Connectors:1X02_TINY
- Q1: value MOSFET-PCHANNELSOT23-3 -> Nfet
- R1, R2, R3: value 100 -> 1k
- R10: value 1k -> 2k
- R11: value 10k --CHECK THIS -> 42.2k
- R12: value 100k -> 10k
- R13: value 270k -> 100
- R14: value 1k -> 100
- R15: value 66.5k -> 100
- R16: value 2k -> 100
- R17: value 10k -> 100
- R18: value 42.2k -> 100
- R4: value 100 -> 270k
- R5: value 100 -> 100k
- R6: value 100 -> 10k --CHECK THIS
- R9: value 1k -> 66.5k
- U1: value MAX31856MUD+ -> ADP2503; device My_IC_Digital:TSSOP14 -> My_IC_Power:DFN300X300X80-11N
- U2: value MAX31856MUD+ -> (none); device My_IC_Digital:TSSOP14 -> My_IC_Power:QFN20
- U3: value MAX31856MUD+ -> ADP1614; device My_IC_Digital:TSSOP14 -> My_IC_Power:DFN300X300X80-11N
- U4: value MCP73871 -> MAX31856MUD+; device My_IC_Power:QFN20 -> My_IC_Digital:TSSOP14
- U5: value ADP2503 -> MAX31856MUD+; device My_IC_Power:DFN300X300X80-11N -> My_IC_Digital:TSSOP14
- U6: value ADP1614 -> MAX31856MUD+; device My_IC_Power:DFN300X300X80-11N -> My_IC_Digital:TSSOP14
- moved Q1 357.4 mm to (47.0, 38.1), turned to 90 degrees
- moved C28 335.4 mm to (33.0, 25.4), turned to 90 degrees
- moved C27 335.2 mm to (33.0, 27.9)
- moved C26 334.6 mm to (36.8, 27.9)
- moved R18 334.5 mm to (35.6, 30.5), turned to 270 degrees
- moved C29 334.2 mm to (32.3, 21.6), turned to 270 degrees
- moved R17 332.3 mm to (38.1, 30.5), turned to 270 degrees
- moved R16 328.6 mm to (47.0, 25.4), turned to 270 degrees
- moved R15 326.5 mm to (49.5, 25.4)
- moved L1 324.3 mm to (71.1, 49.5), turned to 270 degrees
- moved C25 323.9 mm to (41.9, 30.5)
- moved D5 322.6 mm to (31.8, 48.3), turned to 270 degrees
- moved C23 319.7 mm to (53.3, 26.7), turned to 270 degrees
- moved L2 312.0 mm to (25.4, 48.3)
- moved C24 309.5 mm to (41.9, 17.8)
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Connections:
- removed net 6V5_VIN: C26.1, C27.2, L2.1, Q1.2, U6.3, U6.8
- removed net CS_TC_1: U1.9
- removed net CS_TC_2: U2.9
- removed net CS_TC_3: U3.9
- removed net N$24: D5.A-2, L2.2, U6.6, U6.7
- removed net TC+: C1.1, C11.1, C12.2, C2.2, C6.1, C7.2, R2.2, R4.2, R6.2, U1.4, U2.4, U3.4
- removed net TC-: C1.2, C11.2, C13.1, C3.1, C6.2, C8.1, R1.2, R3.2, R5.2, U1.3, U2.3, U3.3
- new net 6V5_INDUCTOR: D5.A-2, L2.2, U3.6, U3.7
- new net BAT_V_EN: Q2.1, U7.1
- new net BAT_V_READ: R22.1, R23.2, U7.22
- new net FLASH_CS: U7.12, U9.1
- new net N$23: ANT1.1, U8.9
- new net N$25: Q2.2, R22.2
- new net N$27: R20.1, U7.23
- new net N$30: C31.1, J6.1
- new net N$31: C19.1, C20.2, R16.2, U5.4
- new net N$32: C18.1, C19.2, R15.2, U5.3
- new net N$33: U7.27
- new net N$34: U7.28
- new net N$35: U7.19
- new net N$36: D7.ANODE, R21.2
- new net N$37: D6.ANODE, R20.2
- new net N$38: C16.1, C17.2, R14.2, U4.4
- new net N$39: C15.1, C16.2, R13.2, U4.3
- new net N$40: C25.1, C26.2, R17.2, U6.3
- new net N$41: C26.1, C27.2, R18.2, U6.4
- new net N$52: U7.8, Y1.3
- new net N$53: U7.7, Y1.1
- new net N$54: C30.1, U7.20
- new net N_SEL1: JP1.2, U7.24
- new net N_SEL2: JP2.2, U7.25
- new net N_SEL3: JP3.2, U7.26
- new net PIN_9: R21.1, U7.13
- new net RF_CS: U7.14, U8.5
- new net RF_INT: U7.32, U8.14
- new net RST: C31.2, R19.2, TC1.P$5, U7.29
- new net RX: J6.3, U7.30
- new net TC1_CS: U4.9, U7.11
- new net TC2_CS: U6.9, U7.10
- new net TC3_CS: U5.9, U7.9
- new net TX: J6.2, U7.31
- net 3V3: now also C2.1, C21.2, C22.2, C23.2, C24.2, C28.2, C29.2, C3.1, J6.4, JP1.1, JP2.1, JP3.1, R19.1, TC1.P$2, U1.1, U1.10, U4.5, U4.8, U5.5, U5.8, U6.5, U6.8, U7.18, U7.4, U7.6, U8.13, U9.3, U9.7, U9.8; no longer C10.2, C14.2, C15.2, C21.1, C22.1, C4.2, C5.2, C9.2, U1.5, U1.8, U2.5, U2.8, U3.5, U3.8, U5.1, U5.10
- net 6V5: now also C13.2, C14.1, J2.NEG, R11.2; no longer C28.2, C29.1, R18.2
- net GND: now also BATT1.NEG_1, BATT1.NEG_2, BATT1.NEG_3, C1.2, C10.2, C11.NEG, C12.2, C13.1, C14.2, C15.2, C17.1, C2.2, C20.1, C21.1, C22.1, C23.1, C24.1, C29.1, C30.2, C4.2, C5.2, C6.1, C7.2, C9.2, D6.CATHODE, D7.CATHODE, J1.NEG, J6.6, Q1.2, R23.1, R24.1, R5.1, R6.1, R9.2, TC1.P$6, U1.11, U1.3, U1.7, U1.9, U2.10, U2.11, U3.11, U3.4, U3.5, U4.1, U4.14, U5.1, U5.14, U6.1, U6.14, U7.21, U7.3, U7.5, U7.PAD, U8.1, U8.10, U8.8, U9.4, Y1.2; no longer BATT1.NEG, C10.1, C12.1, C13.2, C14.1, C15.1, C16.P$2, C17.2, C19.2, C2.1, C20.2, C21.2, C22.2, C23.2, C24.2, C26.2, C29.2, C4.1, C5.1, C7.1, C9.1, J4.SLEEVE1, J4.SLEEVE2, R11.1, R15.2, R17.1, U1.1, U1.14, U2.1, U2.14, U3.1, U3.14, U4.10, U4.11, U5.11, U5.3, U5.7, U5.9, U6.11, U6.4, U6.5
- net HTR_EN: now also R24.2, U3.3, U7.2
- net MISO: now also TC1.P$1, U4.11, U5.11, U6.11, U7.16, U8.2, U9.2; no longer U1.11, U2.11, U3.11
- net MOSI: now also TC1.P$4, U4.12, U5.12, U6.12, U7.15, U8.3, U9.5; no longer U1.12, U2.12, U3.12
- net N$1: now also J5.POS, R18.1; no longer J2.P$1, R4.1
- net N$10: now also D2.CATHODE, U2.7; no longer D3.CATHODE, U4.7
- net N$11: now also D1.CATHODE, U2.8; no longer D4.CATHODE, U4.8
- net N$12: now also R6.2, U2.13; no longer R8.2, U4.13
- net N$13: now also U2.12; no longer U4.12
- net N$14: now also D3.ANODE, R1.1; no longer D2.ANODE, R9.1
- net N$15: now also D2.ANODE, R2.1; no longer D3.ANODE, R10.1
- net N$16: now also D1.ANODE, R3.1; no longer D4.ANODE, R14.1
- net N$17: now also U1.4; no longer U5.4
- net N$18: now also U1.2; no longer U5.2
- net N$19: now also R8.2, U2.5; no longer U4.5
- net N$2: now also J5.NEG, R17.1, U6.2; no longer J2.P$2, R3.1, U2.2
- net N$20: now also J2.POS, Q1.3; no longer R11.2
- net N$21: now also C8.1, U3.10; no longer C25.1, U6.10
- net N$22: now also R9.1, U3.9; no longer R15.1, U6.9
- net N$26: now also R11.1, R12.2, U3.2; no longer R17.2, R18.1, U6.2
- net N$28: now also C10.1, R10.2, U3.1; no longer C24.1, R16.2, U6.1
- net N$29: now also C9.1, R10.1; no longer C23.1, R16.1
- net N$3: now also J4.POS, R16.1; no longer J3.P$1, R6.1
- net N$4: now also J4.NEG, R15.1, U5.2; no longer J3.P$2, R5.1, U3.2
- net N$5: now also D4.A, J1.POS; no longer D1.A, J4.PIN
- net N$6: now also D3.CATHODE, U2.6; no longer D2.CATHODE, U4.6
- net N$7: now also R4.1, R5.2, U2.2; no longer R12.2, R13.1, U4.2
- net N$8: now also J3.POS, R14.1; no longer J1.P$1, R2.1
- net N$9: now also J3.NEG, R13.1, U4.2; no longer J1.P$2, R1.1, U1.2
- net SCK: now also TC1.P$3, U4.10, U5.10, U6.10, U7.17, U8.4, U9.6; no longer U1.10, U2.10, U3.10
- net V_BAT: now also BATT1.POS_1, BATT1.POS_2, BATT1.POS_3, C1.1, C5.1, C6.2, C7.1, L2.1, Q2.3, U1.5, U1.6, U1.8, U2.14, U2.15, U2.16, U3.8; no longer BATT1.POS, C19.1, C20.1, Q1.3, U4.14, U4.15, U4.16, U5.5, U5.6, U5.8
- net V_LOAD: now also C4.1, U2.1, U2.20; no longer C18.1, U4.1, U4.20
- net V_SOLAR: now also C11.POS, C12.1, D4.C, R1.2, R2.2, R3.2, R4.2, U2.17, U2.18, U2.19, U2.3, U2.4, U2.9; no longer C16.P$1, C17.1, D1.C, R10.2, R13.2, R14.2, R9.2, U4.17, U4.18, U4.19, U4.3, U4.4, U4.9
Routing:
- net 3V3: track 0.00 -> 292.3 mm, vias 0 -> 11
- net V_BAT: track 0.00 -> 104.0 mm, vias 0 -> 3
- net V_SOLAR: track 0.00 -> 80.1 mm, vias 0 -> 5
- net HTR_EN: track 0.00 -> 73.0 mm, vias 0 -> 6
- net SCK: track 0.00 -> 64.0 mm, vias 0 -> 3
- net MISO: track 0.00 -> 61.9 mm, vias 0 -> 5
- net MOSI: track 0.00 -> 59.9 mm, vias 0 -> 5
- net BAT_V_EN: track 0.00 -> 59.3 mm, vias 0 -> 4
- net N$5: track 0.00 -> 57.6 mm
- net BAT_V_READ: track 0.00 -> 51.0 mm, vias 0 -> 2
- net N_SEL3: track 0.00 -> 44.4 mm, vias 0 -> 1
- net N_SEL2: track 0.00 -> 41.1 mm, vias 0 -> 1
- net PIN_9: track 0.00 -> 40.8 mm, vias 0 -> 2
- net N_SEL1: track 0.00 -> 40.2 mm, vias 0 -> 1
- net RST: track 0.00 -> 39.7 mm, vias 0 -> 3
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- added copper zone on layer 1, net 6V5_INDUCTOR
- added copper zone on layer 1, net GND
- added copper zone on layer 16, net GND
- added copper zone on layer 1, net V_BAT
- added copper zone on layer 16, net V_BAT
- added copper zone on layer 1, net V_LOAD
- added copper zone on layer 16, net V_SOLAR
Other:
- board size 100 x 80 mm -> 76.2 x 54.6 mm
- board text added: "+"
- board text added: "1"
- board text added: "2"
- board text added: "4"
- board text added: "GND"
- board text added: "Tx"
- board text added: "sap flux v10 2016.12"
- board text added: "v10"
