File: sap-flux/hardware/pcb/sap_flux-v10.sch (EAGLE design)
At the start: 68 parts, among them J1 MF-CON-2.54mm-01x02, J2 MF-CON-2.54mm-01x02, J3 MF-CON-2.54mm-01x02, J4 KLDX-0202-B, Q1 MOSFET-PCHANNELSOT23-3, U1 MAX31856MUD+, U2 MAX31856MUD+, U3 MAX31856MUD+, U4 MCP73871, U5 ADP2503, U6 ADP1614

Commit message: sap flux BOM, Gerbers, Radiation Shield Files
Parts:
- added ANT1: ANTENNA-433_CHIP, My_RF:ANTENNA-433_CHIP
- added C30, C31: 0.1uF, My_Passives:CAPACITOR_NP0603-N
- added D6: green, My_LEDs:LED_SINGLE-0603
- added D7: red, My_LEDs:LED_SINGLE-0603
- added FRAME3: FRAME-LETTERNO_PACKAGE, My_Aesthetics:FRAME-LETTERNO_PACKAGE
- added J5: CON_01X02TINY, My_Connectors:CON_01X02TINY
- added J6: (no value), My_Connectors:ARDUINO_SERIAL_PROGRAMPTH
- added JP1: 1, My_Passives:JUMPER-PAD-2-NOYES_SILK
- added JP2: 2, My_Passives:JUMPER-PAD-2-NOYES_SILK
- added JP3: 4, My_Passives:JUMPER-PAD-2-NOYES_SILK
- added LOGO1: OSHW-LOGOS-COPPER, My_Aesthetics:OSHW-LOGOS-COPPER
- added Q2: battery reading nfet, My_Descrete_Semiconductors:MOSFET-NCHANNELSOT23-3
- added R19, R24: 10k, My_Passives:RESISTOR0603-N
- added R20, R21: 1k, My_Passives:RESISTOR0603-N
- added R22: 33k, My_Passives:RESISTOR0603-N
- added R23: 68k, My_Passives:RESISTOR0603-N
- added TC1: TC2030-IDC-NL, My_Connectors:CON_02X03_AVRISP_TC2030-IDC-NL
- added U7: ATMEGA328P_32PIN-MU, My_IC_Digital:ATMEGA328P_32PIN-MU
- added U8: RFM69HCW-433MHZ, My_RF:RFM69HCW-433MHZ
- added U9: WINBOND_FLASH_4MBIT-SOIC, My_IC_Digital:WINBOND_FLASH_4MBIT-SOIC
- added Y1: 8MHZ, My_xTal:RESONATOR8MHZ
- BATT1: value BATTERY_HOLDER18650 -> BATTERY_HOLDER-18650_CLIP; device My_Connectors:BATTERY_HOLDER18650 -> My_Connectors:BATTERY_HOLDER-18650_CLIP
- C1, C14, C4, C5, C6: value 0.1uF -> 10uF; device My_Passives:CAPACITOR_NP0603-N -> My_Passives:CAPACITOR_NP0805-N; PARTNO (none) -> GRM21BR61C106KE15K
- C10: value 0.1uF -> 3300pF; PARTNO (none) -> C0603C332K4RACTU
- C11: value 0.1uF -> 4700uF; device My_Passives:CAPACITOR_NP0603-N -> My_Passives:CAPACITOR_P-TH_5MM
- C12, C13, C2, C3, C7: value 0.01uF -> 10uF; device My_Passives:CAPACITOR_NP0603-N -> My_Passives:CAPACITOR_NP0805-N; PARTNO (none) -> GRM21BR61C106KE15K
- C15: value 0.1uF -> 0.01uF; PARTNO (none) -> GRM188R71C103KA01D
- C16: value 4700uF -> 0.1uF; device My_Passives:CAPACITOR_P_10MM -> My_Passives:CAPACITOR_NP0603-N; PARTNO (none) -> CC0603KRX7R7BB104
- C17, C18, C20, C27: value 10uF -> 0.01uF; device My_Passives:CAPACITOR_NP0805-N -> My_Passives:CAPACITOR_NP0603-N; PARTNO (none) -> GRM188R71C103KA01D
- C19, C21, C22, C26, C28, C29: value 10uF -> 0.1uF; device My_Passives:CAPACITOR_NP0805-N -> My_Passives:CAPACITOR_NP0603-N; PARTNO (none) -> CC0603KRX7R7BB104
- C23: value 22nF -> 0.1uF; PARTNO (none) -> CC0603KRX7R7BB104
- C24: value 33pF -> 0.1uF; PARTNO (none) -> CC0603KRX7R7BB104
- C25: value 47nF -> 0.01uF; PARTNO (none) -> GRM188R71C103KA01D
- C8: value 0.01uF -> 4700pF; PARTNO (none) -> GRM188R71C472KA01D
- C9: value 0.1uF -> 2200pF; PARTNO (none) -> GRM188R71C222KA01D
- D1: value PMEG4005EJ -> (none); device My_Descrete_Semiconductors:DIODE-SCHOTTKY-PMEG4005EJ -> My_LEDs:LED_SINGLE-0603; PARTNO (none) -> LTST-C191KRKT
- D2, D3: PARTNO (none) -> LTST-C191KRKT
- D4: value (none) -> DIODE-SCHOTTKY-SOD123FL; device My_LEDs:LED_SINGLE-0603 -> My_Descrete_Semiconductors:DIODE-SCHOTTKY-SOD123FL; PARTNO (none) -> MBR120VLSFT1G
- D5: value DIODE-SCHOTTKYSOD128 -> DIODE-SCHOTTKY-SOD128; device My_Descrete_Semiconductors:DIODE-SCHOTTKYSOD128 -> My_Descrete_Semiconductors:DIODE-SCHOTTKY-SOD128; PARTNO (none) -> CMS05(TE12L,Q,M)
- J1: value MF-CON-2.54mm-01x02 -> CON_01X02-0.2"_POL; device My_Connectors:CON_01X02_PTH_2.54MM -> My_Connectors:CON_01X02-0.2"_POL; LABEL01 Tc+ -> (none); LABEL02 Tc- -> (none)
- J2, J3: value MF-CON-2.54mm-01x02 -> CON_01X02TINY; device My_Connectors:CON_01X02_PTH_2.54MM -> My_Connectors:CON_01X02TINY; LABEL01 Tc+ -> (none); LABEL02 Tc- -> (none)
- J4: value KLDX-0202-B -> CON_01X02TINY; device My_Connectors:DC_PWR_JACK_2.5MM_RIGHT -> My_Connectors:CON_01X02TINY; PARTNO FIND THIS PART AND CHECK FOOTPRINT -> (none)
- L1: PARTNO (none) -> NR3015T1R5N
- Q1: value MOSFET-PCHANNELSOT23-3 -> Nfet; PARTNO (none) -> DMN2075U-7
- R1, R2, R3: value 100 -> 1k; PARTNO (none) -> RC0603FR-071KL
- R10: value 1k -> 2k; PARTNO (none) -> RC0603FR-072KL
- R11: value 10k --CHECK THIS -> 42.2k; PARTNO (none) -> RC0603FR-0742K2L
- R12: value 100k -> 10k; PARTNO (none) -> RC0603FR-0710KL
- R13: value 270k -> 100; PARTNO (none) -> RC0603FR-07100RL
- R14: value 1k -> 100; PARTNO (none) -> RC0603FR-07100RL
- R15: value 66.5k -> 100; PARTNO (none) -> RC0603FR-07100RL
- R16: value 2k -> 100; PARTNO (none) -> RC0603FR-07100RL
- R17: value 10k -> 100; PARTNO (none) -> RC0603FR-07100RL
- R18: value 42.2k -> 100; PARTNO (none) -> RC0603FR-07100RL
- R4: value 100 -> 270k; PARTNO (none) -> RC0603FR-07270KL
- R5: value 100 -> 100k; PARTNO (none) -> RC0603FR-07100KL
- R6: value 100 -> 10k --CHECK THIS; PARTNO (none) -> RC0603FR-0710KL
- R7: PARTNO (none) -> RC0603FR-07100KL
- R8: PARTNO (none) -> RC0603FR-0710KL
- R9: value 1k -> 66.5k; PARTNO (none) -> RC0603FR-0766K5L
- U1: value MAX31856MUD+ -> ADP2503; device My_IC_Digital:MAX31856MUD+ -> My_IC_Power:ADP2503; PARTNO (none) -> ADP2503ACPZ-3.3-R7
- U2: value MAX31856MUD+ -> MCP73871; device My_IC_Digital:MAX31856MUD+ -> My_IC_Power:MCP73871
- U3: value MAX31856MUD+ -> ADP1614; device My_IC_Digital:MAX31856MUD+ -> My_IC_Power:ADP1614; PARTNO (none) -> ADP1614ACPZ-650-R7
- U4: value MCP73871 -> MAX31856MUD+; device My_IC_Power:MCP73871 -> My_IC_Digital:MAX31856MUD+
- U5: value ADP2503 -> MAX31856MUD+; device My_IC_Power:ADP2503 -> My_IC_Digital:MAX31856MUD+
- U6: value ADP1614 -> MAX31856MUD+; device My_IC_Power:ADP1614 -> My_IC_Digital:MAX31856MUD+
Connections:
- removed net 6V5_VIN: C26.1, C27.2, L2.P$1, Q1.S, U6.EN, U6.VIN
- removed net CS_TC_1: U1.CS
- removed net CS_TC_2: U2.CS
- removed net CS_TC_3: U3.CS
- removed net N$24: D5.A, L2.P$2, U6.SW
- removed net TC+: C1.1, C11.1, C12.2, C2.2, C6.1, C7.2, R2.P$2, R4.P$2, R6.P$2, U1.T+, U2.T+, U3.T+
- removed net TC-: C1.2, C11.2, C13.1, C3.1, C6.2, C8.1, R1.P$2, R3.P$2, R5.P$2, U1.T-, U2.T-, U3.T-
- new net 6V5_INDUCTOR: D5.A, L2.P$2, U3.SW
- new net BAT_V_EN: Q2.G, U7.PD3(INT1)
- new net BAT_V_READ: R22.P$1, R23.P$2, U7.ADC7
- new net FLASH_CS: U7.PB0(ICP), U9.CS
- new net N$23: ANT1.1, U8.ANT
- new net N$25: Q2.S, R22.P$2
- new net N$27: R20.P$1, U7.PC0(ADC0)
- new net N$30: C31.1, J6.DTR
- new net N$31: C19.1, C20.2, R16.P$2, U5.T+
- new net N$32: C18.1, C19.2, R15.P$2, U5.T-
- new net N$33: U7.PC4(ADC4/SDA)
- new net N$34: U7.PC5(ADC5/SCL)
- new net N$35: U7.ADC6
- new net N$36: D7.ANODE, R21.P$2
- new net N$37: D6.ANODE, R20.P$2
- new net N$38: C16.1, C17.2, R14.P$2, U4.T+
- new net N$39: C15.1, C16.2, R13.P$2, U4.T-
- new net N$40: C25.1, C26.2, R17.P$2, U6.T-
- new net N$41: C26.1, C27.2, R18.P$2, U6.T+
- new net N$52: U7.PB7(XTAL2/TOSC2), Y1.3
- new net N$53: U7.PB6(XTAL1/TOSC1), Y1.1
- new net N$54: C30.1, U7.AREF
- new net N_SEL1: JP1.2, U7.PC1(ADC1)
- new net N_SEL2: JP2.2, U7.PC2(ADC2)
- new net N_SEL3: JP3.2, U7.PC3(ADC3)
- new net PIN_9: R21.P$1, U7.PB1(OC1A)
- new net RF_CS: U7.PB2(SS/OC1B), U8.NSS
- new net RF_INT: U7.PD2(INT0), U8.DIO0
- new net RST: C31.2, R19.P$2, TC1.PIN5, U7.PC6(/RESET)
- new net RX: J6.TXO, U7.PD0(RXD)
- new net TC1_CS: U4.CS, U7.PD7(AIN1)
- new net TC2_CS: U6.CS, U7.PD6(AIN0)
- new net TC3_CS: U5.CS, U7.PD5(T1)
- new net TX: J6.RXI, U7.PD1(TXD)
- net 3V3: now also C2.1, C21.2, C22.2, C23.2, C24.2, C28.2, C29.2, C3.1, J6.VCC, JP1.1, JP2.1, JP3.1, R19.P$1, TC1.PIN2, U1.FB, U1.VOUT, U4.AVDD, U4.DVDD, U5.AVDD, U5.DVDD, U6.AVDD, U6.DVDD, U7.AVCC, U7.VCC@1, U7.VCC@2, U8.3.3V, U9.HLD, U9.VCC, U9.WP; no longer C10.2, C14.2, C15.2, C21.1, C22.1, C4.2, C5.2, C9.2, U1.AVDD, U1.DVDD, U2.AVDD, U2.DVDD, U3.AVDD, U3.DVDD, U5.FB, U5.VOUT
- net 6V5: now also C13.2, C14.1, J2.PIN1, R11.P$2; no longer C28.2, C29.1, R18.P$2
- net GND: now also C1.2, C10.2, C11.NET, C12.2, C13.1, C14.2, C15.2, C17.1, C2.2, C20.1, C21.1, C22.1, C23.1, C24.1, C29.1, C30.2, C4.2, C5.2, C6.1, C7.2, C9.2, D6.CATHODE, D7.CATHODE, J1.PIN1, J6.GND, Q1.S, R23.P$1, R24.P$1, R5.P$1, R6.P$1, R9.P$2, TC1.PIN6, U1.GND, U1.SYNC, U2.GND1, U2.GND2, U3.GND, U4.AGND, U4.DGND, U5.AGND, U5.DGND, U6.AGND, U6.DGND, U7.AGND, U7.GND@1, U7.GND@2, U8.GND@1, U8.GND@2, U9.GND, Y1.2; no longer C10.1, C12.1, C13.2, C14.1, C15.1, C16.P$2, C17.2, C19.2, C2.1, C20.2, C21.2, C22.2, C23.2, C24.2, C26.2, C29.2, C4.1, C5.1, C7.1, C9.1, J4.SLEEVE, J4.SLEEVE_SHUNT, R11.P$1, R15.P$2, R17.P$1, U1.AGND, U1.DGND, U2.AGND, U2.DGND, U3.AGND, U3.DGND, U4.GND1, U4.GND2, U5.GND, U5.SYNC, U6.GND
- net HTR_EN: now also R24.P$2, U3.EN, U7.PD4(XCK/T0)
- net MISO: now also TC1.PIN1, U4.SDO, U5.SDO, U6.SDO, U7.PB4(MISO), U8.MISO, U9.MISO; no longer U1.SDO, U2.SDO, U3.SDO
- net MOSI: now also TC1.PIN4, U4.SDI, U5.SDI, U6.SDI, U7.PB3(MOSI/OC2), U8.MOSI, U9.MOSI; no longer U1.SDI, U2.SDI, U3.SDI
- net N$1: now also J5.PIN2, R18.P$1; no longer J2.PIN1, R4.P$1
- net N$10: now also D2.CATHODE, U2.STAT2; no longer D3.CATHODE, U4.STAT2
- net N$11: now also D1.CATHODE, U2.STAT1/LBO; no longer D4.CATHODE, U4.STAT1/LBO
- net N$12: now also R6.P$2, U2.PROG1; no longer R8.P$2, U4.PROG1
- net N$13: now also U2.PROG3; no longer U4.PROG3
- net N$14: now also D3.ANODE, R1.P$1; no longer D2.ANODE, R9.P$1
- net N$15: now also D2.ANODE, R2.P$1; no longer D3.ANODE, R10.P$1
- net N$16: now also D1.ANODE, R3.P$1; no longer D4.ANODE, R14.P$1
- net N$17: now also U1.SW1; no longer U5.SW1
- net N$18: now also U1.SW2; no longer U5.SW2
- net N$19: now also R8.P$2, U2.THERM; no longer U4.THERM
- net N$2: now also J5.PIN1, R17.P$1, U6.BIAS; no longer J2.PIN2, R3.P$1, U2.BIAS
- net N$20: now also J2.PIN2, Q1.D; no longer R11.P$2
- net N$21: now also C8.1, U3.SS; no longer C25.1, U6.SS
- net N$22: now also R9.P$1, U3.CLRES; no longer R15.P$1, U6.CLRES
- net N$26: now also R11.P$1, R12.P$2, U3.FB; no longer R17.P$2, R18.P$1, U6.FB
- net N$28: now also C10.1, R10.P$2, U3.COMP; no longer C24.1, R16.P$2, U6.COMP
- net N$29: now also C9.1, R10.P$1; no longer C23.1, R16.P$1
- net N$3: now also J4.PIN2, R16.P$1; no longer J3.PIN1, R6.P$1
- net N$4: now also J4.PIN1, R15.P$1, U5.BIAS; no longer J3.PIN2, R5.P$1, U3.BIAS
- net N$5: now also D4.A, J1.PIN2; no longer D1.A, J4.PIN
- net N$6: now also D3.CATHODE, U2./PG; no longer D2.CATHODE, U4./PG
- net N$7: now also R4.P$1, R5.P$2, U2.VPCC; no longer R12.P$2, R13.P$1, U4.VPCC
- net N$8: now also J3.PIN2, R14.P$1; no longer J1.PIN1, R2.P$1
- net N$9: now also J3.PIN1, R13.P$1, U4.BIAS; no longer J1.PIN2, R1.P$1, U1.BIAS
- net SCK: now also TC1.PIN3, U4.SCK, U5.SCK, U6.SCK, U7.PB5(SCK), U8.SCK, U9.CLK; no longer U1.SCK, U2.SCK, U3.SCK
- net V_BAT: now also C1.1, C5.1, C6.2, C7.1, L2.P$1, Q2.D, U1.EN, U1.PVIN, U1.VIN, U2.VBAT1, U2.VBAT2, U2.VBAT3, U3.VIN; no longer C19.1, C20.1, Q1.D, U4.VBAT1, U4.VBAT2, U4.VBAT3, U5.EN, U5.PVIN, U5.VIN
- net V_LOAD: now also C4.1, U2.OUT1, U2.OUT2; no longer C18.1, U4.OUT1, U4.OUT2
- net V_SOLAR: now also C11.POS, C12.1, D4.C, R1.P$2, R2.P$2, R3.P$2, R4.P$2, U2./TE, U2.CE, U2.IN1, U2.IN2, U2.PROG2, U2.SEL; no longer C16.P$1, C17.1, D1.C, R10.P$2, R13.P$2, R14.P$2, R9.P$2, U4./TE, U4.CE, U4.IN1, U4.IN2, U4.PROG2, U4.SEL
Other:
- note added: "3.3v Buck/Boost Reg"
- note added: "6.5v Boost Reg"
- note added: "Batt_V Divider"
- note added: "FTDI In double check Rx/Tx"
- note added: "MCU"
- note added: "Network Selection"
- note added: "PRGM Header"
- note added: "RFM69HCW"
- note added: "SPI Flash"
- note added: "Solar Input"
- note added: "Solar Li Ion Battery Charger"
- note added: "Thermocouple 1"
- note added: "Thermocouple 2"
- note added: "Thermocouple 3"
- note removed: "TEST THIS FIRST!!!! DOES IT WORK?!?!"
