File: datalogger/hardware/pcb/datalogger-v10.brd (EAGLE design)
At the start: 59.7 x 40.6 mm, 42 parts, among them J1 FTDI_DEVICE, J2 U.FL, J4 5.5x2.1mm Barrel, J6 MF-CON-2.54mm-01x03, U1 RFM69HCW, U2 TPS63030DSKT, X1 8MHZ

Commit message: again....this is stupid
Parts:
- removed ATMEGA328: ATMega-328, LowPowerLab:TQFP32-08
- removed J1: FTDI_DEVICE, SparkFun-Connectors:FTDI_DEVICE_SIDE
- removed JP1: USD-SOCKETNEW, SparkFun-Connectors:MICRO-SD-SOCKET-PP
- removed TC1: TC2030-IDC-NL, MF_Connectors:TC2030-IDC-NL
- removed U$3: DS3231M, _my-parts:SO08
- removed U$4: TSP62161, _my-parts:WSON-8
- added J5: MF-CON-2.54mm-01x03, My_Connectors:PTH_2.54MM_01X03
- added JP2: USD-SDIO-SOCKET, My_Connectors:MICRO-SD-SOCKET-SDIO
- added TC2: TC2030-IDC-NL, My_Connectors:TC2030-IDC-NL
- added U4: DS3231M, My_IC_Digital:SO08
- added U5: ATMEGA168/328TQFP32, My_IC_Digital:TQFP32-08
- added U6: TPS62161, My_IC_Power:WSON-8
- J6: value MF-CON-2.54mm-01x03 -> MF-CON-2.54mm-01x06; device MF_Connectors:PTH_2.54MM_01X03 -> My_Connectors:PTH_2.54MM_01X06
- U$1: value BATTERY_HOLDER -> BATTERY_HOLDER12MM
- U2: device Texas Instruments_By_element14_Batch_1:SON50P260X260X80-11N -> My_IC_Power:SON50P260X260X80-11N
- moved J6 105.7 mm to (-26.7, -78.7), turned to 0 degrees
- moved U2 64.1 mm to (-24.1, -43.2), turned to 0 degrees
Connections:
- removed net N$5: J1.P$5
- net 12V_IN: now also J5.P$3, U6.6; no longer J6.P$3, U$4.6
- net A0: now also U5.23; no longer ATMEGA328.23
- net A1: now also U5.24; no longer ATMEGA328.24
- net A2: now also U5.25; no longer ATMEGA328.25
- net A3: now also U5.26; no longer ATMEGA328.26
- net A4_SDA: now also U4.7, U5.27; no longer ATMEGA328.27, U$3.7
- net A5_SCL: now also U4.8, U5.28; no longer ATMEGA328.28, U$3.8
- net A6: now also U5.19; no longer ATMEGA328.19
- net A7: now also U5.22; no longer ATMEGA328.22
- net AREF: now also U5.20; no longer ATMEGA328.20
- net BAT_IN: now also J5.P$1; no longer J6.P$1
- net D0_RX: now also J6.P$2, U5.30; no longer ATMEGA328.30, J1.P$2
- net D10_SS: now also U5.14; no longer ATMEGA328.14
- net D11_MOSI: now also JP2.CMD, TC2.P$3, U5.15; no longer ATMEGA328.15, JP1.DI, TC1.P$4
- net D12_MISO: now also JP2.DAT0, TC2.P$6, U5.16; no longer ATMEGA328.16, JP1.DO, TC1.P$1
- net D13_SCK: now also JP2.CLK, TC2.P$4, U5.17; no longer ATMEGA328.17, JP1.SCLK, TC1.P$3
- net D1_TX: now also J6.P$3, U5.31; no longer ATMEGA328.31, J1.P$3
- net D2_RF-INT: now also U5.32; no longer ATMEGA328.32
- net D3_RTC-INT: now also U4.3, U5.1; no longer ATMEGA328.1, U$3.3
- net D4_CS: now also JP2.CD/DAT3, U5.2; no longer ATMEGA328.2, JP1.CS
- net D5_CD: now also JP2.CD1, JP2.CD2, U5.9; no longer ATMEGA328.9, JP1.CD1, JP1.CD2
- net D6: now also U5.10; no longer ATMEGA328.10
- net D7: now also U5.11; no longer ATMEGA328.11
- net D8: now also U5.12; no longer ATMEGA328.12
- net D9: now also U5.13; no longer ATMEGA328.13
- net GND: now also J6.P$6, JP2.GND, JP2.GND1, JP2.GND3, TC2.P$1, U4.5, U5.21, U5.3, U5.5, U6.1, U6.4, U6.5, U6.P$9; no longer ATMEGA328.21, ATMEGA328.3, ATMEGA328.5, J1.P$6, JP1.GND, JP1.GND1, JP1.GND3, TC1.P$6, U$3.5, U$4.1, U$4.4, U$4.5, U$4.P$9
- net N$1: now also U5.7; no longer ATMEGA328.7
- net N$10: now also U4.6; no longer U$3.6
- net N$13: now also JP2.DAT1; no longer JP1.RSV2
- net N$18: now also U6.8; no longer U$4.8
- net N$21: now also U5.8; no longer ATMEGA328.8
- net N$3: now also JP2.DAT2; no longer JP1.RSV1
- net N$4: now also J6.P$1; no longer J1.P$1
- net RST: now also TC2.P$2, U5.29; no longer ATMEGA328.29, TC1.P$5
- net SW: now also U6.7; no longer U$4.7
- net VCC: now also J5.P$2, J6.P$4, JP2.VCC, TC2.P$5, U4.2, U5.18, U5.4, U5.6; no longer ATMEGA328.18, ATMEGA328.4, ATMEGA328.6, J1.P$4, J6.P$2, JP1.VCC, TC1.P$2, U$3.2
- net V_12V: now also U6.2, U6.3; no longer U$4.2, U$4.3
Routing:
- net D4_CS: track 31.4 -> 0.00 mm, vias 2 -> 0
- net D5_CD: track 28.9 -> 0.00 mm, vias 2 -> 0
- net D1_TX: track 28.8 -> 0.00 mm
- net VCC: track 138.3 -> 111.3 mm
- net D0_RX: track 26.4 -> 0.00 mm
- net RST: track 42.6 -> 19.9 mm, vias 4 -> 2
- net D3_RTC-INT: track 20.5 -> 0.00 mm, vias 2 -> 0
- net V_BAT: track 19.6 -> 12.6 mm
- net BAT_IN: track 4.88 -> 0.02 mm, vias 2 -> 0
- net GND: track 4.21 -> 0.00 mm, vias 4 -> 5
- net D12_MISO: track 33.1 -> 29.7 mm
- net A5_SCL: track 18.0 -> 14.7 mm
- net N$4: track 4.05 -> 1.05 mm
- net D13_SCK: track 34.2 -> 31.5 mm
- net 3V3L2: track 2.68 -> 0.00 mm
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