File: datalogger/hardware/pcb/datalogger-v10.sch (EAGLE design)
At the start: 42 parts, among them J1 FTDI_DEVICE, J2 U.FL, J4 5.5x2.1mm Barrel, J6 MF-CON-2.54mm-01x03, U1 RFM69HCW, U2 TPS63030DSKT, X1 8MHZ

Commit message: again....this is stupid
Parts:
- removed ATMEGA328: ATMega-328, LowPowerLab:ATMEGA168/328TQFP32
- removed J1: FTDI_DEVICE, SparkFun-Connectors:FTDI_DEVICE
- removed JP1: USD-SOCKETNEW, SparkFun-Connectors:USD-SOCKETNEW
- removed TC1: TC2030-IDC-NL, MF_Connectors:CON_02X03_AVRISP_TC2030-IDC-NL
- removed U$3: DS3231M, _my-parts:DS3231M
- removed U$4: TSP62161, _my-parts:TSP62161
- added J5: MF-CON-2.54mm-01x03, My_Connectors:CON_01X03_PTH_2.54MM
- added JP2: USD-SDIO-SOCKET, My_Connectors:USD-SDIO-SOCKET
- added TC2: TC2030-IDC-NL, My_Connectors:CON_02X03_AVRISP_TC2030-IDC-NL
- added U4: DS3231M, My_IC_Digital:DS3231M
- added U5: ATMEGA168/328TQFP32, My_IC_Digital:ATMEGA168/328TQFP32
- added U6: TPS62161, My_IC_Power:TPS62161
- J6: value MF-CON-2.54mm-01x03 -> MF-CON-2.54mm-01x06; device MF_Connectors:CON_01X03_PTH_2.54MM -> My_Connectors:CON_01X06_PTH_2.54MM; LABEL01 Li-Ion -> gnd; LABEL02 VCC -> tx; LABEL03 12v-16v -> rx; LABEL04 (none) -> vcc; LABEL06 (none) -> gnd
- U$1: value BATTERY_HOLDER -> BATTERY_HOLDER12MM; device Custom_Parts:BATTERY_HOLDER -> Custom_Parts:BATTERY_HOLDER12MM
- U2: device Texas Instruments_By_element14_Batch_1:TPS63030DSKT -> My_IC_Power:TPS63030DSKT
Connections:
- removed net N$5: J1.CTS
- net 12V_IN: now also J5.PIN3, U6.VOS; no longer J6.PIN3, U$4.VOS
- net A0: now also U5.PC0(ADC0); no longer ATMEGA328.PC0(ADC0)
- net A1: now also U5.PC1(ADC1); no longer ATMEGA328.PC1(ADC1)
- net A2: now also U5.PC2(ADC2); no longer ATMEGA328.PC2(ADC2)
- net A3: now also U5.PC3(ADC3); no longer ATMEGA328.PC3(ADC3)
- net A4_SDA: now also U4.SDA, U5.PC4(ADC4/SDA); no longer ATMEGA328.PC4(ADC4/SDA), U$3.SDA
- net A5_SCL: now also U4.SCL, U5.PC5(ADC5/SCL); no longer ATMEGA328.PC5(ADC5/SCL), U$3.SCL
- net A6: now also U5.ADC6; no longer ATMEGA328.ADC6
- net A7: now also U5.ADC7; no longer ATMEGA328.ADC7
- net AREF: now also U5.AREF; no longer ATMEGA328.AREF
- net BAT_IN: now also J5.PIN1; no longer J6.PIN1
- net D0_RX: now also J6.PIN2, U5.PD0(RXD); no longer ATMEGA328.PD0(RXD), J1.TXO
- net D10_SS: now also U5.PB2(SS/OC1B); no longer ATMEGA328.PB2(SS/OC1B)
- net D11_MOSI: now also JP2.CMD, TC2.PIN3, U5.PB3(MOSI/OC2); no longer ATMEGA328.PB3(MOSI/OC2), JP1.DI, TC1.PIN4
- net D12_MISO: now also JP2.DAT0, TC2.PIN6, U5.PB4(MISO); no longer ATMEGA328.PB4(MISO), JP1.DO, TC1.PIN1
- net D13_SCK: now also JP2.CLK, TC2.PIN4, U5.PB5(SCK); no longer ATMEGA328.PB5(SCK), JP1.SCK, TC1.PIN3
- net D1_TX: now also J6.PIN3, U5.PD1(TXD); no longer ATMEGA328.PD1(TXD), J1.RXI
- net D2_RF-INT: now also U5.PD2(INT0); no longer ATMEGA328.PD2(INT0)
- net D3_RTC-INT: now also U4.INT, U5.PD3(INT1); no longer ATMEGA328.PD3(INT1), U$3.INT
- net D4_CS: now also JP2.CD/DAT3, U5.PD4(XCK/T0); no longer ATMEGA328.PD4(XCK/T0), JP1.CS
- net D5_CD: now also JP2.CD1, JP2.CD2, U5.PD5(T1); no longer ATMEGA328.PD5(T1), JP1.CD1, JP1.CD2
- net D6: now also U5.PD6(AIN0); no longer ATMEGA328.PD6(AIN0)
- net D7: now also U5.PD7(AIN1); no longer ATMEGA328.PD7(AIN1)
- net D8: now also U5.PB0(ICP); no longer ATMEGA328.PB0(ICP)
- net D9: now also U5.PB1(OC1A); no longer ATMEGA328.PB1(OC1A)
- net GND: now also J6.PIN6, JP2.GND, JP2.SHIELD@1, JP2.SHIELD@3, TC2.PIN1, U4.GND, U5.AGND, U5.GND@1, U5.GND@2, U6.AGND, U6.FB, U6.PGND; no longer ATMEGA328.AGND, ATMEGA328.GND@1, ATMEGA328.GND@2, J1.GND, JP1.GND, JP1.SHIELD@1, JP1.SHIELD@3, TC1.PIN6, U$3.GND, U$4.AGND, U$4.FB, U$4.PGND
- net N$1: now also U5.PB6(XTAL1/TOSC1); no longer ATMEGA328.PB6(XTAL1/TOSC1)
- net N$10: now also U4.VBAT; no longer U$3.VBAT
- net N$13: now also JP2.DAT1; no longer JP1.RSV
- net N$18: now also U6.PG; no longer U$4.PG
- net N$21: now also U5.PB7(XTAL2/TOSC2); no longer ATMEGA328.PB7(XTAL2/TOSC2)
- net N$3: now also JP2.DAT2; no longer JP1.NC
- net N$4: now also J6.PIN1; no longer J1.DTR
- net RST: now also TC2.PIN2, U5.PC6(/RESET); no longer ATMEGA328.PC6(/RESET), TC1.PIN5
- net SW: now also U6.SW; no longer U$4.SW
- net VCC: now also J5.PIN2, J6.PIN4, JP2.VCC, TC2.PIN5, U4.VCC, U5.AVCC, U5.VCC@1, U5.VCC@2; no longer ATMEGA328.AVCC, ATMEGA328.VCC@1, ATMEGA328.VCC@2, J1.VCC, J6.PIN2, JP1.VCC, TC1.PIN2, U$3.VCC
- net V_12V: now also U6.EN, U6.VIN; no longer U$4.EN, U$4.VIN
Other:
- moved on the sheet: C1, C10, C11, C5, J2, R1, SJ1, SJ2, SJ3, SJ4, SJ5, SJ6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
