File: datalogger/logger-v20/hardware/pcb/datalogger-v21.brd (EAGLE design)
At the start: 76.2 x 64.8 mm, 68 parts, among them J10 MF-CON-2.54mm-01x03, J11 MF-CON-2.54mm-01x02, J2 U.FL, J3 CON_01X02SCREW_0.2", J4 ANTENNA_SMA_EDGE, J5 MF-CON-2.54mm-01x03, J6 MF-CON-2.54mm-01x03, J7 MF-CON-2.54mm-01x03, J8 MF-CON-2.54mm-01x03, J9 MF-CON-2.54mm-01x03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

Commit message: small changes to datalogger
Parts:
- removed R14: 10k, My_Passives:R0603-N
- added C11: 0.1uF, My_Passives:C0603-N
Connections:
- net 3V3: no longer R14.1, SJ1.1, SJ2.1, SJ3.1
- net GND: now also C11.2, SJ1.1, SJ2.1, SJ3.1
- net RAIN_INT: now also C11.1; no longer R14.2
Routing:
- net 3V3: track 236.2 -> 222.2 mm
- net GND: track 0.00 -> 5.08 mm
- net RAIN_INT: track 45.1 -> 45.9 mm
Changed lines of the file:
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@@
 <?xml version="1.0" encoding="utf-8"?>
 <!DOCTYPE eagle SYSTEM "eagle.dtd">
-<eagle version="8.0.0">
+<eagle version="8.0.1">
 <drawing>
 <settings>
@@
 <attribute name="NAME" x="11.66" y="46.97" size="0.7" layer="25" font="vector" ratio="11" rot="R270"/>
 </element>
-<element name="R14" library="My_Passives" package="R0603-N" value="10k" x="12.7" y="44.45" smashed="yes" rot="R270">
-<attribute name="PARTNO" value="" x="12.7" y="44.45" size="1.778" layer="27" font="vector" ratio="15" rot="R270" display="off"/>
-<attribute name="NAME" x="13.599078125" y="46.00890625" size="0.7" layer="25" font="vector" ratio="11" rot="R270"/>
+<element name="C11" library="My_Passives" package="C0603-N" value="0.1uF" x="13.97" y="44.45">
+<attribute name="PARTNO" value="" x="13.97" y="44.45" size="1.778" layer="27" font="vector" ratio="15" display="off"/>
 </element>
 </elements>
@@
 <via x="20.955" y="44.45" extent="1-16" drill="0.381"/>
 <via x="39.116" y="39.624" extent="1-16" drill="0.381"/>
+<contactref element="SJ1" pad="1"/>
+<contactref element="SJ2" pad="1"/>
+<contactref element="SJ3" pad="1"/>
+<wire x1="43.18" y1="42.36" x2="40.64" y2="42.36" width="0.3048" layer="1"/>
+<wire x1="40.64" y1="42.36" x2="38.1" y2="42.36" width="0.3048" layer="1"/>
+<contactref element="C11" pad="2"/>
 </signal>
 <signal name="RST">
@@
 <contactref element="TC1" pad="P$2"/>
 <contactref element="U4" pad="2"/>
-<contactref element="SJ1" pad="1"/>
-<contactref element="SJ2" pad="1"/>
-<contactref element="SJ3" pad="1"/>
 <contactref element="R4" pad="2"/>
 <contactref element="R3" pad="2"/>
@@
 <contactref element="Q4" pad="1"/>
 <contactref element="R11" pad="2"/>
-<contactref element="R14" pad="1"/>
 <wire x1="64.516" y1="23.914" x2="64.3" y2="24.13" width="0.3048" layer="1"/>
-<wire x1="43.18" y1="42.36" x2="40.64" y2="42.36" width="0.3048" layer="1"/>
-<wire x1="40.64" y1="42.36" x2="38.1" y2="42.36" width="0.3048" layer="1"/>
 <wire x1="40.29" y1="31.75" x2="39.497" y2="31.75" width="0.3048" layer="1"/>
 <wire x1="39.497" y1="31.75" x2="39.116" y2="32.131" width="0.3048" layer="1"/>
@@
 <wire x1="11.938" y1="61.341" x2="11.938" y2="62.192" width="0.3048" layer="1"/>
 <wire x1="11.938" y1="62.192" x2="11.9" y2="62.23" width="0.3048" layer="1"/>
-<wire x1="12.7" y1="45.25" x2="20.612" y2="45.25" width="0.4064" layer="1"/>
 <wire x1="21.463" y1="54.356" x2="21.59" y2="54.483" width="0.4064" layer="1"/>
 <wire x1="21.59" y1="54.483" x2="21.717" y2="54.61" width="0.4064" layer="1"/>
@@
 <wire x1="16.383" y1="57.15" x2="18.923" y2="57.15" width="0.4064" layer="1"/>
 <wire x1="18.923" y1="57.15" x2="21.59" y2="54.483" width="0.4064" layer="1"/>
-<wire x1="38.1" y1="42.36" x2="37.026" y2="42.36" width="0.4064" layer="1"/>
 <wire x1="37.026" y1="42.36" x2="36.576" y2="41.91" width="0.4064" layer="1"/>
 <wire x1="36.576" y1="41.91" x2="36.576" y2="40.818" width="0.4064" layer="1"/>
@@
 <signal name="RAIN_INT">
 <contactref element="J11" pad="P$2"/>
-<contactref element="R14" pad="2"/>
 <contactref element="U3" pad="11"/>
-<wire x1="12.7" y1="43.65" x2="12.23" y2="43.18" width="0.3048" layer="1"/>
-<wire x1="12.23" y1="43.18" x2="10.16" y2="43.18" width="0.3048" layer="1"/>
 <wire x1="38.29" y1="25.75" x2="38.29" y2="26.987" width="0.3048" layer="1"/>
 <wire x1="38.29" y1="26.987" x2="38.481" y2="27.178" width="0.3048" layer="1"/>
@@
 <wire x1="29.083" y1="26.797" x2="27.305" y2="26.797" width="0.3048" layer="1"/>
 <wire x1="27.305" y1="26.797" x2="22.225" y2="31.877" width="0.3048" layer="1"/>
-<wire x1="22.225" y1="31.877" x2="22.225" y2="41.783" width="0.3048" layer="1"/>
-<wire x1="22.225" y1="41.783" x2="20.32" y2="43.688" width="0.3048" layer="1"/>
-<wire x1="20.32" y1="43.688" x2="12.738" y2="43.688" width="0.3048" layer="1"/>
-<wire x1="12.738" y1="43.688" x2="12.7" y2="43.65" width="0.3048" layer="1"/>
+<wire x1="22.225" y1="41.783" x2="22.225" y2="31.877" width="0.3048" layer="1"/>
 <wire x1="29.083" y1="26.797" x2="31.496" y2="29.21" width="0.3048" layer="1"/>
 <wire x1="31.496" y1="29.21" x2="37.084" y2="29.21" width="0.3048" layer="1"/>
 <wire x1="37.084" y1="29.21" x2="38.481" y2="27.813" width="0.3048" layer="1"/>
+<contactref element="C11" pad="1"/>
+<wire x1="20.828" y1="43.18" x2="22.225" y2="41.783" width="0.3048" layer="1"/>
+<wire x1="13.17" y1="43.18" x2="10.16" y2="43.18" width="0.3048" layer="1"/>
+<wire x1="13.17" y1="43.18" x2="20.828" y2="43.18" width="0.3048" layer="1"/>
+<wire x1="13.17" y1="44.45" x2="13.17" y2="43.18" width="0.3048" layer="1"/>
 </signal>
 </signals>
