File: datalogger/logger-v20/hardware/pcb/datalogger-v21.sch (EAGLE design)
At the start: 68 parts, among them J10 MF-CON-2.54mm-01x03, J11 MF-CON-2.54mm-01x02, J2 U.FL, J3 CON_01X02SCREW_0.2", J4 ANTENNA_SMA_EDGE, J5 MF-CON-2.54mm-01x03, J6 MF-CON-2.54mm-01x03, J7 MF-CON-2.54mm-01x03, J8 MF-CON-2.54mm-01x03, J9 MF-CON-2.54mm-01x03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

Commit message: ...
Parts:
- J1: device My_Connectors:USB-5PINMICRO_STRONG -> My_Connectors:USB-5PIN_B-MICRO_R/A_STRONG
- J8: LABEL01 (none) -> -; LABEL02 (none) -> data; LABEL03 (none) -> +
Connections:
- net NET_SEL_4: now also U3.PC3(TMS); no longer U3.PD6(PWM)
- net RF_CS: now also U3.PC2(TCK); no longer U3.PB4(PWM/SS)
- net SD_LED_0: now also U3.PD6(PWM); no longer U3.PC2(TCK)
- net SD_LED_1: now also U3.PB4(PWM/SS); no longer U3.PC3(TMS)
Changed lines of the file:
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@@
 </part>
 <part name="U2" library="My_IC_Digital" deviceset="FT232RL-BASIC" device="-SSOP"/>
-<part name="J1" library="My_Connectors" deviceset="USB-5PIN" device="MICRO_STRONG"/>
+<part name="J1" library="My_Connectors" deviceset="USB-5PIN" device="_B-MICRO_R/A_STRONG"/>
 <part name="C1" library="My_Passives" deviceset="CAPACITOR_NP" device="0603-N" value="0.1uF"/>
 <part name="C2" library="My_Passives" deviceset="CAPACITOR_NP" device="0603-N" value="0.1uF"/>
@@
 <part name="J6" library="My_Connectors" deviceset="CON_01X03" device="_PTH_2.54MM" value="MF-CON-2.54mm-01x03"/>
 <part name="J7" library="My_Connectors" deviceset="CON_01X03" device="_PTH_2.54MM" value="MF-CON-2.54mm-01x03"/>
-<part name="J8" library="My_Connectors" deviceset="CON_01X03" device="_PTH_2.54MM" value="MF-CON-2.54mm-01x03"/>
+<part name="J8" library="My_Connectors" deviceset="CON_01X03" device="_PTH_2.54MM" value="MF-CON-2.54mm-01x03">
+<attribute name="LABEL01" value="-"/>
+<attribute name="LABEL02" value="data"/>
+<attribute name="LABEL03" value="+"/>
+</part>
 <part name="D6" library="My_LEDs" deviceset="LED_SINGLE" device="-0603"/>
 <part name="R13" library="My_Passives" deviceset="RESISTOR" device="0603-N" value="680"/>
@@
 </segment>
 <segment>
-<wire x1="177.8" y1="144.78" x2="180.34" y2="144.78" width="0.1524" layer="91"/>
-<label x="180.34" y="144.78" size="1.27" layer="95" xref="yes"/>
-<pinref part="U3" gate="G$1" pin="PB4(PWM/SS)"/>
+<wire x1="132.08" y1="129.54" x2="129.54" y2="129.54" width="0.1524" layer="91"/>
+<label x="129.54" y="129.54" size="1.27" layer="95" rot="R180" xref="yes"/>
+<pinref part="U3" gate="G$1" pin="PC2(TCK)"/>
 </segment>
 </net>
@@
 <net name="NET_SEL_4" class="0">
 <segment>
-<wire x1="177.8" y1="119.38" x2="180.34" y2="119.38" width="0.1524" layer="91"/>
-<label x="180.34" y="119.38" size="1.27" layer="95" xref="yes"/>
-<pinref part="U3" gate="G$1" pin="PD6(PWM)"/>
-</segment>
-<segment>
 <pinref part="SJ1" gate="G$1" pin="2"/>
 <wire x1="236.22" y1="160.02" x2="236.22" y2="157.48" width="0.1524" layer="91"/>
 <label x="236.22" y="157.48" size="1.27" layer="95" rot="R270" xref="yes"/>
 </segment>
-</net>
-<net name="SD_LED_1" class="0">
 <segment>
 <wire x1="132.08" y1="127" x2="129.54" y2="127" width="0.1524" layer="91"/>
@@
 <pinref part="U3" gate="G$1" pin="PC3(TMS)"/>
 </segment>
+</net>
+<net name="SD_LED_1" class="0">
 <segment>
 <pinref part="R9" gate="G$1" pin="P$1"/>
 <wire x1="55.88" y1="83.82" x2="53.34" y2="83.82" width="0.1524" layer="91"/>
 <label x="53.34" y="83.82" size="1.27" layer="95" rot="R270" xref="yes"/>
+</segment>
+<segment>
+<wire x1="177.8" y1="144.78" x2="180.34" y2="144.78" width="0.1524" layer="91"/>
+<label x="180.34" y="144.78" size="1.27" layer="95" xref="yes"/>
+<pinref part="U3" gate="G$1" pin="PB4(PWM/SS)"/>
 </segment>
 </net>
@@
 <net name="SD_LED_0" class="0">
 <segment>
-<wire x1="132.08" y1="129.54" x2="129.54" y2="129.54" width="0.1524" layer="91"/>
-<label x="129.54" y="129.54" size="1.27" layer="95" rot="R180" xref="yes"/>
-<pinref part="U3" gate="G$1" pin="PC2(TCK)"/>
-</segment>
-<segment>
 <pinref part="R10" gate="G$1" pin="P$1"/>
 <wire x1="12.7" y1="83.82" x2="10.16" y2="83.82" width="0.1524" layer="91"/>
 <label x="10.16" y="83.82" size="1.27" layer="95" rot="R270" xref="yes"/>
 </segment>
-</net>
+<segment>
+<wire x1="177.8" y1="119.38" x2="180.34" y2="119.38" width="0.1524" layer="91"/>
+<label x="180.34" y="119.38" size="1.27" layer="95" xref="yes"/>
+<pinref part="U3" gate="G$1" pin="PD6(PWM)"/>
+</segment>
+</net>

Commit message: small changes to datalogger
Parts:
- removed R14: 10k, My_Passives:RESISTOR0603-N
- added C11: 0.1uF, My_Passives:CAPACITOR_NP0603-N
Connections:
- net 3V3: no longer R14.P$1, SJ1.1, SJ2.1, SJ3.1
- net GND: now also C11.2, SJ1.1, SJ2.1, SJ3.1
- net RAIN_INT: now also C11.1; no longer R14.P$2
Other:
- moved on the sheet: SW1
Changed lines of the file:
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@@
 <?xml version="1.0" encoding="utf-8"?>
 <!DOCTYPE eagle SYSTEM "eagle.dtd">
-<eagle version="7.7.0">
+<eagle version="8.0.1">
 <drawing>
 <settings>
@@
 <part name="J10" library="My_Connectors" deviceset="CON_01X03" device="_PTH_2.54MM" value="MF-CON-2.54mm-01x03"/>
 <part name="J11" library="My_Connectors" deviceset="CON_01X02" device="_PTH_2.54MM" value="MF-CON-2.54mm-01x02"/>
-<part name="R14" library="My_Passives" deviceset="RESISTOR" device="0603-N" value="10k"/>
+<part name="C11" library="My_Passives" deviceset="CAPACITOR_NP" device="0603-N" value="0.1uF"/>
 </parts>
 <sheets>
@@
 <instance part="C13" gate="G$1" x="127" y="76.2"/>
 <instance part="TC1" gate="G$1" x="53.34" y="58.42" rot="R180"/>
-<instance part="SW1" gate="G$1" x="223.52" y="132.08"/>
+<instance part="SW1" gate="G$1" x="220.98" y="124.46"/>
 <instance part="Y1" gate="G$1" x="121.92" y="152.4"/>
 <instance part="Q1" gate="G$1" x="17.78" y="17.78" rot="MR270"/>
@@
 <segment>
 <pinref part="SW1" gate="G$1" pin="P$3"/>
-<wire x1="220.98" y1="129.54" x2="220.98" y2="127" width="0.1524" layer="91"/>
-<wire x1="220.98" y1="127" x2="223.52" y2="127" width="0.1524" layer="91"/>
+<wire x1="218.44" y1="121.92" x2="218.44" y2="119.38" width="0.1524" layer="91"/>
+<wire x1="218.44" y1="119.38" x2="220.98" y2="119.38" width="0.1524" layer="91"/>
 <pinref part="SW1" gate="G$1" pin="P$4"/>
-<wire x1="223.52" y1="127" x2="226.06" y2="127" width="0.1524" layer="91"/>
-<wire x1="226.06" y1="127" x2="226.06" y2="129.54" width="0.1524" layer="91"/>
-<wire x1="223.52" y1="127" x2="223.52" y2="121.92" width="0.1524" layer="91"/>
-<label x="223.52" y="121.92" size="1.27" layer="95" rot="R270" xref="yes"/>
+<wire x1="220.98" y1="119.38" x2="223.52" y2="119.38" width="0.1524" layer="91"/>
+<wire x1="223.52" y1="119.38" x2="223.52" y2="121.92" width="0.1524" layer="91"/>
+<wire x1="220.98" y1="119.38" x2="220.98" y2="114.3" width="0.1524" layer="91"/>
+<label x="220.98" y="114.3" size="1.27" layer="95" rot="R270" xref="yes"/>
 </segment>
 <segment>
@@
 <label x="30.48" y="10.16" size="1.27" layer="95" rot="R270" xref="yes"/>
 </segment>
+<segment>
+<pinref part="SJ1" gate="G$1" pin="1"/>
+<wire x1="236.22" y1="170.18" x2="236.22" y2="172.72" width="0.1524" layer="91"/>
+<wire x1="236.22" y1="172.72" x2="228.6" y2="172.72" width="0.1524" layer="91"/>
+<pinref part="SJ2" gate="G$1" pin="1"/>
+<wire x1="228.6" y1="172.72" x2="228.6" y2="170.18" width="0.1524" layer="91"/>
+<wire x1="228.6" y1="172.72" x2="220.98" y2="172.72" width="0.1524" layer="91"/>
+<pinref part="SJ3" gate="G$1" pin="1"/>
+<wire x1="220.98" y1="172.72" x2="220.98" y2="170.18" width="0.1524" layer="91"/>
+<label x="220.98" y="172.72" size="1.27" layer="95" rot="R180" xref="yes"/>
+</segment>
 </net>
 <net name="RST" class="0">
@@
 <segment>
 <pinref part="SW1" gate="G$1" pin="P$2"/>
-<wire x1="226.06" y1="134.62" x2="226.06" y2="137.16" width="0.1524" layer="91"/>
-<wire x1="226.06" y1="137.16" x2="223.52" y2="137.16" width="0.1524" layer="91"/>
+<wire x1="223.52" y1="127" x2="223.52" y2="129.54" width="0.1524" layer="91"/>
+<wire x1="223.52" y1="129.54" x2="220.98" y2="129.54" width="0.1524" layer="91"/>
 <pinref part="SW1" gate="G$1" pin="P$1"/>
-<wire x1="223.52" y1="137.16" x2="220.98" y2="137.16" width="0.1524" layer="91"/>
-<wire x1="220.98" y1="137.16" x2="220.98" y2="134.62" width="0.1524" layer="91"/>
-<wire x1="223.52" y1="137.16" x2="223.52" y2="142.24" width="0.1524" layer="91"/>
-<label x="223.52" y="142.24" size="1.27" layer="95" rot="R90" xref="yes"/>
+<wire x1="220.98" y1="129.54" x2="218.44" y2="129.54" width="0.1524" layer="91"/>
+<wire x1="218.44" y1="129.54" x2="218.44" y2="127" width="0.1524" layer="91"/>
+<wire x1="220.98" y1="129.54" x2="220.98" y2="134.62" width="0.1524" layer="91"/>
+<label x="220.98" y="134.62" size="1.27" layer="95" rot="R90" xref="yes"/>
 </segment>
 <segment>
@@
 <label x="68.58" y="152.4" size="1.27" layer="95" xref="yes"/>
 <pinref part="U4" gate="G$1" pin="VCC"/>
-</segment>
-<segment>
-<pinref part="SJ1" gate="G$1" pin="1"/>
-<wire x1="236.22" y1="170.18" x2="236.22" y2="172.72" width="0.1524" layer="91"/>
-<wire x1="236.22" y1="172.72" x2="228.6" y2="172.72" width="0.1524" layer="91"/>
-<pinref part="SJ2" gate="G$1" pin="1"/>
-<wire x1="228.6" y1="172.72" x2="228.6" y2="170.18" width="0.1524" layer="91"/>
-<wire x1="228.6" y1="172.72" x2="220.98" y2="172.72" width="0.1524" layer="91"/>
-<pinref part="SJ3" gate="G$1" pin="1"/>
-<wire x1="220.98" y1="172.72" x2="220.98" y2="170.18" width="0.1524" layer="91"/>
-<label x="220.98" y="172.72" size="1.27" layer="95" rot="R180" xref="yes"/>
 </segment>
 <segment>
@@
 <instance part="J10" gate="G$1" x="109.22" y="147.32" rot="R180"/>
 <instance part="J11" gate="G$1" x="111.76" y="124.46" rot="R180"/>
-<instance part="R14" gate="G$1" x="116.84" y="132.08"/>
+<instance part="C11" gate="G$1" x="124.46" y="119.38"/>
 </instances>
 <busses>
@@
 <label x="116.84" y="124.46" size="1.27" layer="95" rot="R270" xref="yes"/>
 </segment>
+<segment>
+<pinref part="C11" gate="G$1" pin="2"/>
+<wire x1="124.46" y1="114.3" x2="124.46" y2="111.76" width="0.1524" layer="91"/>
+<label x="124.46" y="111.76" size="1.27" layer="95" rot="R270" xref="yes"/>
+</segment>
 </net>
 <net name="N$23" class="0">
@@
 <label x="17.78" y="170.18" size="1.27" layer="95" rot="R90" xref="yes"/>
 </segment>
-<segment>
-<pinref part="R14" gate="G$1" pin="P$1"/>
-<wire x1="111.76" y1="132.08" x2="109.22" y2="132.08" width="0.1524" layer="91"/>
-<wire x1="109.22" y1="132.08" x2="109.22" y2="134.62" width="0.1524" layer="91"/>
-<label x="109.22" y="134.62" size="1.27" layer="95" rot="R90" xref="yes"/>
-</segment>
 </net>
 <net name="N$13" class="0">
@@
 <wire x1="114.3" y1="127" x2="124.46" y2="127" width="0.1524" layer="91"/>
 <label x="129.54" y="127" size="1.27" layer="95" xref="yes"/>
-<pinref part="R14" gate="G$1" pin="P$2"/>
+<pinref part="C11" gate="G$1" pin="1"/>
 <wire x1="124.46" y1="127" x2="129.54" y2="127" width="0.1524" layer="91"/>
-<wire x1="121.92" y1="132.08" x2="124.46" y2="132.08" width="0.1524" layer="91"/>
-<wire x1="124.46" y1="132.08" x2="124.46" y2="127" width="0.1524" layer="91"/>
-</segment>
-</net>
+<wire x1="124.46" y1="121.92" x2="124.46" y2="127" width="0.1524" layer="91"/>
+</segment>
+</net>
