File: dendrometer/dendro-v20/hardware/pcb/add-ons/sensor_sunstone.sch (EAGLE design)
At the start: 28 parts, among them J1 AVR_SPI_PRG_6PTH, Q2 MOSFET-P, U1 ATMEGA328P, U2 LM4040A20IDBZT

Commit message: working on updating code and building add-on mods for system
Parts:
- removed J1: AVR_SPI_PRG_6PTH, SparkFun-Connectors:AVR_SPI_PRG_6PTH
- removed JP2: M01PTH, SparkFun-Connectors:M01PTH
- removed R8: 330, passives-7351:RESISTOR0603-N
- removed U$2: TPS61097-33, _my-parts:TPS61097-33
- removed U$4: 4.7uH, _my-parts:INDUCTORS_WURTH
- removed U$6: MCP3426A0-E/SN, Microchip_By_element14_Batch_1:MCP3426A0-E/SN
- added ANT: M01PTH, SparkFun-Connectors:M01PTH
- added ICSP: AVR_SPI_PRG_6PTH, SparkFun-Connectors:AVR_SPI_PRG_6PTH
- added U3: MCP3425A0T-E/CH, Microchip_By_element14_Batch_1:MCP3425A0T-E/CH
- added U4: INDUCTORS_WURTH, _my-parts:INDUCTORS_WURTH
- Q2: value MOSFET-P -> PFET
- R3: value 1M -> 2M
- R4: value 10k -> DNP
- R6: value 480 -> 10k
- R7: value THERM -> 5.9k
- U2: value LM4040A20IDBZT -> TPS61097-33; device Texas Instruments_By_element14_Batch_1:LM4040A20IDBZT -> _my-parts:TPS61097-33
Connections:
- removed net SENS: SENS.2, U$6.CH1+
- removed net S_EN: Q2.D, R8.P$1
- removed net THERM: R4.P$2, R7.P$1, U$6.CH2+
- removed net V_REF: R4.P$1, R8.P$2, SENS.3, U2.CATHODE
- new net N$2: Q2.D, R4.P$2, R7.P$2
- new net N$6: SENS.2, U3.VIN+
- new net V-EXCITE: R4.P$1, R7.P$1, SENS.3, U1.PC1(ADC1)
- net GND: now also ICSP.6, U2.GND, U3.VIN-, U3.VSS; no longer J1.6, R7.P$2, U$2.GND, U$6.CH1-, U$6.CH2-, U$6.VSS, U2.ANODE
- net MISO: now also ICSP.1; no longer J1.1
- net MOSI: now also ICSP.4; no longer J1.4
- net N$1: now also U2.L, U4.P$1; no longer U$2.L, U$4.P$1
- net N$7: now also ANT.1; no longer JP2.1
- net RST: now also ICSP.5; no longer J1.5
- net SCK: now also ICSP.3; no longer J1.3
- net SCL: now also U3.SCL; no longer U$6.SCL
- net SDA: now also U3.SDA; no longer U$6.SDA
- net V3.3: now also ICSP.2, U2.VOUT, U3.VDD; no longer J1.2, U$2.VOUT, U$6.VDD
- net VBAT: now also U2.EN, U2.VIN, U4.P$2; no longer U$2.EN, U$2.VIN, U$4.P$2
Other:
- note removed: "ADC"
- note removed: "HEADERS"
- note removed: "MCU"
- note removed: "POWER"
- note removed: "RADIO"
- note removed: "V_REF"
- note removed: "switch to 61097A"
- moved on the sheet: C1, C2, C3, C4, C5, C6, C7, LED1, PGRM, Q2, R1, R2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
